File: eagle/controllerHat/controllerHat.brd (EAGLE design)
At the start: 43.2 x 49.5 mm, 46 parts, among them J4 USB-MICROB

Commit message: bulk commit (eagle files, old changes)
Parts:
- removed H1, H2, H3, H4: MOUNT-HOLE2.8, holes:2,8
- removed ICSP2: (no value), SparkFun-Connectors:2X3
- removed J3: (no value), SparkFun-Connectors:1X02_LOCK
- removed R2, R3: (no value), SparkFun-Passives:1206
- removed R5: 36k, SparkFun-Passives:1206
- removed R6: 3k, SparkFun-Passives:1206
- removed R7: 2k, SparkFun-Passives:1206
- removed T_CAM1, T_CAM2: (no value), SparkFun-DiscreteSemi:TO-92
- removed U$2: (no value), adafruit:CR2032-SMD
- U$1: value DS3234 -> PIZERO_THROUGH_HOLE; device SparkFun-FreqCtrl:DS3234 -> pizero:PIZERO_THOUGH_HOLE
- moved U$1 58.5 mm to (0.00, 0.00), turned to 0 degrees
- moved RTC1 39.9 mm to (50.0, 5.08), turned to 180 degrees
- moved Q2 35.6 mm to (12.7, 3.81), turned to 180 degrees
- moved J5 29.2 mm to (20.3, 3.81), turned to 0 degrees
- moved R1 28.1 mm to (14.0, 7.62), turned to 0 degrees
- moved R9 25.4 mm to (43.2, 2.54)
- moved SH 23.6 mm to (20.7, 10.2)
- moved T_ZERO1 23.0 mm to (14.0, 10.2), turned to 0 degrees
- moved C2 21.6 mm to (61.0, 21.6)
- moved J4 21.6 mm to (62.6, 15.2)
- moved RUSB1 21.6 mm to (57.1, 12.7)
- moved RUSB2 21.6 mm to (57.1, 17.8)
- moved J1 20.3 mm to (55.9, 5.08)
- moved R8 19.2 mm to (36.8, 2.54)
- moved C3 19.1 mm to (58.4, 8.89)
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Connections:
- removed net N$12: R6.2, R7.1, T_CAM1.3, T_CAM2.1
- removed net N$13: R5.2, R6.1, T_CAM2.3
- removed net N$18: R2.2, T_CAM1.2
- removed net N$19: R3.2, T_CAM2.2
- removed net N$6: J3.2, R5.1, T_CAM1.1
- net CAM1: no longer R2.1
- net CAM2: no longer R3.1
- net GND: no longer ICSP2.4, J3.1, R7.2
- net RST: no longer ICSP2.6
- net RX: no longer ICSP2.3
- net TX: no longer ICSP2.5
- net VCC: no longer ICSP2.2
- net ZERO_EN: no longer ICSP2.1
Routing:
- net CAM_EN: track 6.47 -> 55.5 mm, vias 0 -> 2
- net CELL1: track 13.1 -> 62.0 mm
- net TX: track 38.3 -> 0.00 mm, vias 1 -> 0
- net RST: track 38.1 -> 0.00 mm
- net GND: track 213.7 -> 250.3 mm, vias 2 -> 1
- net RX: track 31.4 -> 0.00 mm, vias 1 -> 0
- net ZERO_EN: track 20.1 -> 0.00 mm
- net GNDA: track 13.2 -> 33.1 mm, vias 0 -> 1
- net N$6: track 16.9 -> 0.00 mm
- net CELL2: track 15.0 -> 29.9 mm, vias 0 -> 2
- net N$13: track 14.0 -> 0.00 mm
- net VD_DIRECT: track 12.7 -> 25.1 mm
- net N$20: track 7.82 -> 20.0 mm
- net VCC: track 111.5 -> 99.5 mm
- net N$8: track 9.55 -> 21.0 mm
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Other:
- board size 43.2 x 49.5 mm -> 64.8 x 49.5 mm
- board text removed: "BOX"
- board text removed: "TIME"
