File: eagle/controllerHat/controllerHat.sch (EAGLE design)
At the start: 46 parts, among them J4 USB-MICROB, Q2 MOSFET-PCHANNELNDP6020P_20V_2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

Commit message: bulk commit (eagle files, old changes)
Parts:
- removed H1, H2, H3, H4: MOUNT-HOLE2.8, holes:MOUNT-HOLE2.8
- removed ICSP2: (no value), SparkFun-Connectors:M03X2FEMALE
- removed J3: (no value), SparkFun-Connectors:M02LOCK
- removed R2, R3: (no value), SparkFun-Passives:RESISTOR1206
- removed R5: 36k, SparkFun-Passives:RESISTOR1206
- removed R6: 3k, SparkFun-Passives:RESISTOR1206
- removed R7: 2k, SparkFun-Passives:RESISTOR1206
- removed T_CAM1, T_CAM2: (no value), SparkFun-DiscreteSemi:TRANSISTOR_NPN2N3904
- removed U$2: (no value), adafruit:CR2032SMT
- U$1: value DS3234 -> PIZERO_THROUGH_HOLE; device SparkFun-FreqCtrl:DS3234 -> pizero:PIZERO_THROUGH_HOLE
Connections:
- removed net N$12: R6.2, R7.1, T_CAM1.C, T_CAM2.E
- removed net N$13: R5.2, R6.1, T_CAM2.C
- removed net N$18: R2.2, T_CAM1.B
- removed net N$19: R3.2, T_CAM2.B
- removed net N$6: J3.2, R5.1, T_CAM1.E
- net CAM1: no longer R2.1
- net CAM2: no longer R3.1
- net GND: no longer ICSP2.4, J3.1, R7.2
- net RST: no longer ICSP2.6
- net RX: no longer ICSP2.3
- net TX: no longer ICSP2.5
- net VCC: no longer ICSP2.2
- net ZERO_EN: no longer ICSP2.1
