File: eagle/controllerM2/controllerM2.brd (EAGLE design)
At the start: 55.9 x 44.5 mm, 42 parts, among them U1 ATMEGA328P, X1 1501_04

Commit message: eagle files
Parts:
- removed PWR_BATT, PWR_CAM: (no value), SparkFun-Connectors:POWER_JACK_PTH_BREAD
- removed SHTR: (no value), SparkFun-Connectors:1X03_LOCK
- removed X1: 1501_04, con-lumberg:1501_05
- added J1: (no value), SparkFun-Connectors:1X02_LOCK
- added J3, J4: (no value), SparkFun-Connectors:SCREWTERMINAL-3.5MM-2_LOCK
- added R4: 36k, SparkFun-Resistors:AXIAL-0.3
- added R5: 3k, SparkFun-Resistors:AXIAL-0.3
- added R8: 2k, SparkFun-Resistors:AXIAL-0.3
- moved J2 13.1 mm to (2.54, 15.2)
- moved T_HSS 7.18 mm to (14.0, 25.4), turned to 90 degrees
- moved SH 7.18 mm to (7.62, 23.2)
- moved T_CAM2 4.02 mm to (16.5, 10.2)
- moved HIGHSIDESWITCH 3.59 mm to (14.0, 33.0)
- moved R3 2.54 mm to (31.8, 2.54)
- moved T_CAM1 2.54 mm to (16.5, 16.5), turned to 270 degrees
- moved C1 1.27 mm to (41.9, 2.54)
- moved R6 1.27 mm to (25.4, 20.3)
- moved R7 1.27 mm to (25.4, 17.8)
- moved VD21 1.27 mm to (25.4, 27.9)
- moved ZERO 1.27 mm to (51.7, 36.8)
- moved DISP 1.27 mm to (8.89, 5.08)
- moved R1 1.27 mm to (27.9, 7.62)
- moved R10 1.27 mm to (27.9, 33.0)
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Connections:
- removed net N$10: SHTR.3, T_CAM1.3, X1.3
- new net N$16: R4.P$1, R5.P$2, T_CAM1.1
- new net N$17: R5.P$1, R8.P$2, T_CAM2.1
- net BATT_VCC: now also J4.2; no longer PWR_BATT.PWR
- net CAM_OUT: now also J3.2; no longer PWR_CAM.PWR
- net GND: now also J1.1, R8.P$1; no longer SHTR.1, T_CAM1.1, T_CAM2.1, X1.1
- net GNDA: now also J3.1, J4.1; no longer PWR_BATT.GND, PWR_CAM.GND
- net N$7: now also J1.2, R4.P$2, T_CAM1.3; no longer SHTR.2, X1.2
Routing:
- net TX: track 78.1 -> 46.7 mm, vias 0 -> 2
- net N$16: track 0.00 -> 15.4 mm
- net GND: track 175.4 -> 160.7 mm, vias 0 -> 1
- net N$10: track 14.7 -> 0.00 mm
- net N$5: track 9.54 -> 22.4 mm
- net N$2: track 6.78 -> 19.6 mm
- net N$7: track 11.7 -> 24.2 mm
- net CELL1: track 35.0 -> 23.1 mm, vias 0 -> 1
- net N$13: track 6.60 -> 16.0 mm
- net N$17: track 0.00 -> 8.08 mm
- net GNDA: track 20.1 -> 12.6 mm
- net SDA: track 38.4 -> 31.8 mm
- net CAM_OUT: track 17.6 -> 11.3 mm
- net CELL2: track 23.5 -> 28.2 mm, vias 1 -> 0
- net VCC: track 81.3 -> 77.9 mm
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Other:
- board size 55.9 x 44.5 mm -> 54.6 x 44.5 mm
- board text added: "M"

Commit message: bulk commit (eagle files, old changes)
Parts:
- moved CONV_X_VCC 1.27 mm to (31.8, 41.9)
- moved R3 1.27 mm to (33.0, 2.54)
- moved TEMP 1.27 mm to (36.8, 41.9)
Routing:
- net VCC: track 77.9 -> 99.2 mm
- net TX: track 46.7 -> 52.2 mm
- net SDA: track 31.8 -> 28.0 mm
- net N$1: track 7.57 -> 6.30 mm
- net GND: track 160.7 -> 161.4 mm
- net TEMP: track 21.3 -> 21.9 mm
- net BATT_VCC: track 30.1 -> 29.5 mm
