File: eagle/zeroport/zeroport.brd (EAGLE design)
At the start: 20.3 x 55.9 mm, 16 parts, among them Q1 check_pins

Commit message: eagle files
Parts:
- moved J1 48.3 mm to (19.1, 3.81), turned to 90 degrees
- moved J2 48.3 mm to (16.5, 3.81), turned to 90 degrees
- moved R4 19.1 mm to (7.62, 44.5)
- moved T_SHIFTER1 11.5 mm to (10.2, 21.6)
- moved R2 10.2 mm to (7.62, 47.0)
- moved ZERO 7.62 mm to (5.08, 39.4)
- moved R3 5.24 mm to (11.4, 12.7), turned to 90 degrees
- moved R6 5.24 mm to (8.89, 12.7)
- moved T_SHIFTER2 4.58 mm to (3.81, 25.4)
- moved R1 4.58 mm to (8.89, 30.5)
- moved R5 2.54 mm to (5.08, 17.8)
- moved R7 2.54 mm to (2.54, 17.8)
- moved J3 1.27 mm to (8.89, 3.81), turned to 0 degrees
- moved Q1 1.27 mm to (3.81, 8.89), turned to 0 degrees
Routing:
- net GND: track 108.2 -> 54.4 mm, vias 1 -> 0
- net +5V: track 69.7 -> 18.9 mm
- net ZTX: track 48.0 -> 0.00 mm
- net RST: track 36.4 -> 75.6 mm, vias 0 -> 1
- net ZRX: track 38.4 -> 71.7 mm, vias 1 -> 0
- net N$6: track 8.19 -> 23.2 mm
- net MCTX: track 6.13 -> 15.2 mm
- net ZERO_EN: track 29.8 -> 21.0 mm, vias 0 -> 1
- net VCC: track 56.2 -> 64.4 mm
- net N$5: track 22.5 -> 30.7 mm
- net MCRX: track 26.4 -> 20.8 mm
- net N$4: track 4.15 -> 5.43 mm
Other:
- board size 20.3 x 55.9 mm -> 22.9 x 55.9 mm

Commit message: bulk commit (eagle files, old changes)
Parts:
- H1, H2: value MOUNT-HOLE3.2 -> MOUNT-HOLE2.8; device holes:3,2 -> holes:2,8
- R1, R2, R3, R4, R5, R6, R7: device SparkFun-Resistors:AXIAL-0.3 -> SparkFun-Resistors:AXIAL-0.4
- moved R4 10.2 mm to (7.62, 34.3)
- moved R1 6.48 mm to (7.62, 36.8)
- moved R2 3.81 mm to (11.4, 47.0), turned to 270 degrees
- moved ZERO 2.84 mm to (6.35, 41.9), turned to 90 degrees
- moved T_SHIFTER2 2.54 mm to (3.81, 27.9)
- moved H2 1.80 mm to (2.54, 53.3)
- moved H1 1.80 mm to (2.54, 2.54)
- moved T_SHIFTER1 1.80 mm to (11.4, 22.9)
- moved R5 1.27 mm to (5.08, 19.1)
- moved R7 1.27 mm to (2.54, 19.1)
Routing:
- net RST: track 75.6 -> 0.00 mm, vias 1 -> 0
- net ZRX: track 71.7 -> 0.00 mm
- net VCC: track 64.4 -> 0.00 mm
- net GND: track 54.4 -> 0.00 mm
- net N$5: track 30.7 -> 0.00 mm
- net N$6: track 23.2 -> 0.00 mm
- net ZERO_EN: track 21.0 -> 0.00 mm, vias 1 -> 0
- net MCRX: track 20.8 -> 0.00 mm
- net +5V: track 18.9 -> 0.00 mm
- net MCTX: track 15.2 -> 0.00 mm
- net N$4: track 5.43 -> 0.00 mm
- net N$2: track 3.67 -> 0.00 mm
Other:
- board size 22.9 x 55.9 mm -> 24.1 x 55.9 mm
- board text removed: "BOX"
- board text removed: "TIME"
