File: eagle/controllercap/controllercap.sch (EAGLE design)
At the start: 3 parts

Commit message: minor changes
Parts:
- added H1, H2: MOUNT-HOLE2.8, holes:MOUNT-HOLE2.8
Changed lines of the file:
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@@
 <?xml version="1.0" encoding="utf-8"?>
 <!DOCTYPE eagle SYSTEM "eagle.dtd">
-<eagle version="7.6.0">
+<eagle version="7.7.0">
 <drawing>
 <settings>
@@
 <part name="GND16" library="supply1" deviceset="GNDA" device=""/>
 <part name="GND8" library="supply1" deviceset="GNDA" device=""/>
+<part name="H1" library="holes" deviceset="MOUNT-HOLE" device="2.8"/>
+<part name="H2" library="holes" deviceset="MOUNT-HOLE" device="2.8"/>
 </parts>
 <sheets>
@@
 <instance part="GND16" gate="1" x="172.72" y="99.06" rot="R90"/>
 <instance part="GND8" gate="1" x="139.7" y="91.44"/>
+<instance part="H1" gate="G$1" x="124.46" y="60.96"/>
+<instance part="H2" gate="G$1" x="149.86" y="60.96"/>
 </instances>
 <busses>
