File: eagle/controller5Teensy/controller5Teensy.sch (EAGLE design)
At the start: 62 parts, among them Q1 MMBT4403, Q2 FDD4141TO252, U1 LM75AIM, U3 mp2307, U4 ATSAMD21G-A, X1 ZX62D-B-5PA8, X2 ZX62D-B-5PA8, X3 ZX62D-B-5PA8

Commit message: controller5 & controller5Teensy
Parts:
- removed C12: 1uF, SparkFun-Capacitors:CAP1206
- removed C13, C14: 22pF, SparkFun-Passives:CAP1206
- removed C3: 10uF, SparkFun-Passives:CAP1206
- removed RRST, RUSB1, RUSB2: (no value), SparkFun-Passives:RESISTOR1206
- removed U4: ATSAMD21G-A, SparkFun-DigitalIC:ATSAMD21G-A
- removed X2: ZX62D-B-5PA8, zx62d-b-5pa8-oshpark_10:ZX62D-B-5PA8
- removed Y2: (no value), SparkFun-FreqCtrl:CRYSTALCRYSTAL-SMD-5X3-16MHZ
- added J7: (no value), SparkFun-Connectors:M24
Connections:
- removed net D+: RUSB2.1, U4.PA25(SER3:3+)
- removed net D-: RUSB1.1, U4.PA24(SER3:2+)
- removed net MISO: U4.PA12(I2C/SER2:0+)
- removed net MOSI: U4.PB10(SER4:2+)
- removed net N$10: RUSB1.2, X2G$1.2
- removed net N$11: RUSB2.2, X2G$1.3
- removed net N$2: U4.PA30(SWCLK/SER1:2+)
- removed net N$25: C12.2, U4.VDDCORE
- removed net N$27: C13.2, U4.PA00(XIN32/SER1:0/TC2:0), Y2.2
- removed net N$28: C14.2, U4.PA01(XOUT32/SER1:1/TC2:1), Y2.1
- removed net N$3: U4.PA31(SWDIO/SER1:3+)
- removed net RST: RRST.1, U4.!RESET!
- removed net RX: U4.PB23(SER5:3+)
- removed net SCK: U4.PB11(SER4:3+)
- removed net TX: U4.PB22(SER5:2+)
- net GND: no longer C12.1, C13.1, C14.1, C3.2, U4.GND@18, U4.GND@35, U4.GND@42, U4.GNDANA, X2G$1.5
- net N$22: no longer C3.1, X2G$1.1
- net SCL: no longer U4.PA23(I2C/SER3:0+)
- net SDA: no longer U4.PA22(I2C/SER3:0+)
- net VCC: no longer RRST.2, U4.VDDANA, U4.VDDIN, U4.VDDIO@17, U4.VDDIO@36
