File: eagle/controller5/controller5.brd (EAGLE design)
At the start: 53.3 x 64.8 mm, 63 parts, among them Q1 MMBT4403, U1 LM75AIM, U3 mp2307, U4 ATSAMD21G-A, X2 ZX62D-B-5PA8

Commit message: various eagle layouts
Parts:
- added J7: CORTEX_DEBUGPTH, SparkFun-Connectors:2X5-PTH-1.27MM
- added TP1, TP2: TPTP20R, testpad:TP20R
- moved RUSB1 65.6 mm to (66.0, 55.9)
- moved C3 64.9 mm to (66.0, 49.5)
- moved X2 64.9 mm to (55.9, 53.3)
- moved RUSB2 63.8 mm to (64.8, 52.1)
- moved D2 30.7 mm to (61.0, 27.9)
- moved R7 16.7 mm to (11.4, 6.35), turned to 270 degrees
- moved C6 16.5 mm to (16.5, 2.54), turned to 0 degrees
- moved R4 15.3 mm to (21.6, 2.54), turned to 0 degrees
- moved R6 13.7 mm to (11.4, 11.4), turned to 90 degrees
- moved C12 12.0 mm to (45.7, 30.5), turned to 270 degrees
- moved C7 11.7 mm to (21.6, 5.08), turned to 180 degrees
- moved D1 11.4 mm to (14.0, 22.9)
- moved R18 11.4 mm to (23.4, 33.8)
- moved SH1 11.4 mm to (6.35, 25.4)
- moved VD6 11.4 mm to (20.3, 41.9)
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Connections:
- net GND: now also J7.3, J7.5
- net N$2: now also TP1.TP
- net N$3: now also TP2.TP
- net VCC: now also J7.1
Other:
- board size 53.3 x 64.8 mm -> 48.3 x 64.8 mm
