File: eagle/controller5/controller5.sch (EAGLE design)
At the start: 62 parts, among them Q1 MMBT4403, Q2 FDD4141TO252, U1 LM75AIM, U3 mp2307, U4 ATSAMD21G-A, X1 ZX62D-B-5PA8, X2 ZX62D-B-5PA8, X3 ZX62D-B-5PA8

Commit message: various eagle layouts
Parts:
- added J7: CORTEX_DEBUGPTH, SparkFun-Connectors:CORTEX_DEBUGPTH
- added TP1, TP2: TPTP20R, testpad:TPTP20R
Connections:
- net GND: now also J7.GND@3, J7.GND@5
- net N$2: now also TP1.TP
- net N$3: now also TP2.TP
- net VCC: now also J7.VCC
Changed lines of the file:
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@@
 <part name="GND5" library="SparkFun-Aesthetics" deviceset="GND" device=""/>
 <part name="J2" library="SparkFun-Connectors" deviceset="M03" device="LOCK"/>
+<part name="J7" library="SparkFun-Connectors" deviceset="CORTEX_DEBUG" device="PTH"/>
+<part name="SUPPLY2" library="SparkFun-Aesthetics" deviceset="VCC" device=""/>
+<part name="GND10" library="SparkFun-Aesthetics" deviceset="GND" device=""/>
+<part name="TP1" library="testpad" deviceset="TP" device="TP20R"/>
+<part name="TP2" library="testpad" deviceset="TP" device="TP20R"/>
 </parts>
 <sheets>
@@
 <instance part="GND5" gate="1" x="129.54" y="220.98"/>
 <instance part="J2" gate="J$1" x="99.06" y="241.3"/>
+<instance part="J7" gate="G$1" x="223.52" y="144.78"/>
+<instance part="SUPPLY2" gate="G$1" x="203.2" y="152.4"/>
+<instance part="GND10" gate="1" x="198.12" y="144.78" rot="R270"/>
+<instance part="TP1" gate="G$1" x="160.02" y="99.06" rot="R270"/>
+<instance part="TP2" gate="G$1" x="160.02" y="96.52" rot="R270"/>
 </instances>
 <busses>
@@
 <wire x1="228.6" y1="86.36" x2="228.6" y2="91.44" width="0.1524" layer="91"/>
 <pinref part="SUPPLY5" gate="G$1" pin="VCC"/>
+</segment>
+<segment>
+<pinref part="J7" gate="G$1" pin="VCC"/>
+<pinref part="SUPPLY2" gate="G$1" pin="VCC"/>
+<wire x1="208.28" y1="149.86" x2="203.2" y2="149.86" width="0.1524" layer="91"/>
+<wire x1="203.2" y1="149.86" x2="203.2" y2="152.4" width="0.1524" layer="91"/>
 </segment>
 </net>
@@
 <pinref part="GND5" gate="1" pin="GND"/>
 </segment>
+<segment>
+<pinref part="GND10" gate="1" pin="GND"/>
+<wire x1="200.66" y1="144.78" x2="205.74" y2="144.78" width="0.1524" layer="91"/>
+<wire x1="205.74" y1="144.78" x2="205.74" y2="147.32" width="0.1524" layer="91"/>
+<pinref part="J7" gate="G$1" pin="GND@3"/>
+<wire x1="205.74" y1="147.32" x2="208.28" y2="147.32" width="0.1524" layer="91"/>
+<pinref part="J7" gate="G$1" pin="GND@5"/>
+<wire x1="208.28" y1="144.78" x2="205.74" y2="144.78" width="0.1524" layer="91"/>
+<junction x="205.74" y="144.78"/>
+</segment>
 </net>
 <net name="CAM_OUT" class="2">
@@
 <segment>
 <pinref part="U4" gate="G$1" pin="PA30(SWCLK/SER1:2+)"/>
-<wire x1="116.84" y1="99.06" x2="152.4" y2="99.06" width="0.1524" layer="91"/>
-<label x="152.4" y="99.06" size="1.778" layer="95"/>
+<wire x1="116.84" y1="99.06" x2="157.48" y2="99.06" width="0.1524" layer="91"/>
+<pinref part="TP1" gate="G$1" pin="TP"/>
 </segment>
 </net>
@@
 <segment>
 <pinref part="U4" gate="G$1" pin="PA31(SWDIO/SER1:3+)"/>
-<wire x1="116.84" y1="96.52" x2="152.4" y2="96.52" width="0.1524" layer="91"/>
-<label x="152.4" y="96.52" size="1.778" layer="95"/>
-</segment>
-</net>
+<wire x1="116.84" y1="96.52" x2="157.48" y2="96.52" width="0.1524" layer="91"/>
+<pinref part="TP2" gate="G$1" pin="TP"/>
+</segment>
+</net>
