File: eagle/controller6/controller6.sch (EAGLE design)
At the start: 38 parts, among them Q2 FDD4141TO252, U1 LM75AIM, X2 ZX62D-B-5PA8

Commit message: controller6: buck converter
Parts:
- removed CONV_X_VCC: (no value), SparkFun-Connectors:M05LOCK
- removed D1: 1N4004, adafruit:1N4004
- removed J10: (no value), SparkFun-Connectors:M02LOCK
- removed TP1: TPB1,27, testpad:TPB1,27
- added 100K, R1, R4: 6.8k, SparkFun-Resistors:RESISTOR1206
- added C10, C16, C17, C9: 22uF / 6.3V, SparkFun-Capacitors:CAP1206
- added C11, C12, C18, C19: 10uF / 25V, SparkFun-Capacitors:CAP1206
- added C13, C6: 10nF, SparkFun-Capacitors:CAP1206
- added C14, C7: 3.9nF, SparkFun-Capacitors:CAP1206
- added C15, C8: 0.1uF, SparkFun-Capacitors:CAP1206
- added J5: (no value), SparkFun-Connectors:M02PTH
- added L1, L2: 10uH / 4A, SparkFun-Passives:INDUCTORSDR0403-560KL
- added R2, R6: 10k / 1%, SparkFun-Resistors:RESISTOR1206
- added R3: 44k / 1%, SparkFun-Resistors:RESISTOR1206
- added R7: 26.1k / 1%, SparkFun-Resistors:RESISTOR1206
- added U2, U3: MP2307, SparkFun-AnalogIC:GENERIC-SOIC8MSGEQ7N-FILTER
- added X1: ZX62D-B-5PA8, zx62d-b-5pa8-oshpark_10:ZX62D-B-5PA8
Connections:
- removed net N$16: D1.A, Q2.D
- removed net ZERO_EN: U$3.PB7(OC0A/OC1C/RTS)
- removed net ZRX: J3.9
- removed net ZTX: J3.7
- new net BUCK_EN: U$3.PB7(OC0A/OC1C/RTS), U3.7
- new net CONV_3.3V: C10.2, C9.2, L1.1, R7.2, S2.O
- new net N$12: J5.2, X1G$1.3
- new net N$14: C8.2, U2.8
- new net N$15: X1G$1.1
- new net N$17: C6.2, L1.2, U2.3
- new net N$2: 100K.2, U2.7
- new net N$21: C7.1, R4.1
- new net N$23: C7.2, U2.6
- new net N$24: R6.1, R7.1, U2.5
- new net N$25: C15.2, U3.8
- new net N$26: C13.2, L2.2, U3.3
- new net N$27: C13.1, U3.1
- new net N$28: C14.1, R1.1
- new net N$29: C14.2, U3.6
- new net N$3: C6.1, U2.1
- new net N$30: R2.1, R3.1, U3.5
- new net N$37: C18.1, C19.2, U3.2
- new net N$6: J5.1, X1G$1.2
- net +5V: no longer J10.1
- net BATT_VCC: now also 100K.1, C11.1, C12.2, U2.2; no longer CONV_X_VCC.3
- net CAM_OUT: now also Q2.D; no longer D1.C
- net CONV_5V: now also C16.2, C17.2, L2.1, R3.2; no longer CONV_X_VCC.1, S2.O
- net GND: now also C10.1, C11.2, C12.1, C15.1, C16.1, C17.1, C18.2, C19.1, C8.1, C9.1, R1.2, R2.2, R4.2, R6.2, U2.4, U2.PAD, U3.4, U3.PAD, X1G$1.5; no longer CONV_X_VCC.2, TP1.TP
- net RX: now also J3.7
- net TX: now also J3.9
- net VCC: no longer J10.2
Other:
- note added: "5V über mosfet"
- note removed: "PI ZERO MOSFET"
- moved on the sheet: VD5, VD6

Commit message: controller6: multiport connector
Parts:
- removed C1: 100nF, SparkFun-Passives:CAP1206
- removed R17: 10k, SparkFun-Resistors:RESISTOR1206
- removed R18: 1k, SparkFun-Resistors:RESISTOR1206
- removed T_HSS: (no value), SparkFun-DiscreteSemi:TRANSISTOR_NPN2N3904
- removed X1: ZX62D-B-5PA8, zx62d-b-5pa8-oshpark_10:ZX62D-B-5PA8
- added BTS428L2: VOLTAGE_REGULATOR_TLE4476, to252:VOLTAGE_REGULATOR_TLE4476
- added Q1, Q3, Q4: MOSFET-NCHANNELBSS138, SparkFun-DiscreteSemi:MOSFET-NCHANNELBSS138
- added R10, R11, R12, R13, R14: (no value), SparkFun-Passives:RESISTOR0805-RES
- added R5: (no value), SparkFun-Passives:RESISTOR1206
- added S1: TAC_SWITCHSMD, SparkFun-Retired:TAC_SWITCHSMD
- 100K, R1, R2, R3, R4, R6, R7: device SparkFun-Resistors:RESISTOR1206 -> SparkFun-Resistors:RESISTOR0805-RES
- C14, C15, C7, C8: device SparkFun-Capacitors:CAP1206 -> SparkFun-Capacitors:CAP0805
- C3: device SparkFun-Passives:CAP1206 -> SparkFun-Passives:CAP0805
- J2: device SparkFun-Connectors:M04LOCK -> SparkFun-Connectors:M04X2
- Q2: value FDD4141TO252 -> MOSFET-NCHANNELBSS138; device transistor-fet:FDD4141TO252 -> SparkFun-DiscreteSemi:MOSFET-NCHANNELBSS138
- RUSB1, RUSB2: device SparkFun-Passives:RESISTOR1206 -> SparkFun-Passives:RESISTOR0805-RES
Connections:
- removed net +5V: J3.1
- removed net BTN_C: U$3.PF0(ADC0)
- removed net CONV_3.3V: C10.2, C9.2, L1.1, R7.2, S2.O
- removed net N$12: J5.2, X1G$1.3
- removed net N$15: X1G$1.1
- removed net N$36: Q2.G, R17.2, T_HSS.C
- removed net N$37: C18.1, C19.2, U3.2
- new net BTN: R5.2, S1.3, U$3.PF0(ADC0)
- new net CAM3: Q3.G, R12.2
- new net CAM4: Q4.G, R13.1
- new net CONV_3.3_INPUT: 100K.1, C11.1, C12.2, S2.P, U2.2
- new net N$16: J2.2, Q4.D, R13.2
- new net N$18: Q4.S, R14.2
- new net N$32: J2.3, Q2.D, R11.1
- new net N$33: J2.5, Q3.D, R12.1
- new net N$39: BTS428L2.ST
- net BATT_VCC: now also BTS428L2.TAB, C18.1, C19.2, S2.O, U3.2; no longer 100K.1, C11.1, C12.2, Q2.S, R17.1, U2.2
- net CAM1: now also Q1.G, R10.2
- net CAM2: now also Q2.G, R11.2
- net CAM_EN: now also BTS428L2.IN; no longer R18.1
- net CAM_OUT: now also BTS428L2.OUT; no longer Q2.D
- net CONV_5V: now also J3.1
- net GND: now also BTS428L2.GND, J2.7, Q1.S, Q2.S, Q3.S, R14.1, S1.1; no longer T_HSS.E, X1G$1.5
- net N$1: now also J2.4, J5.1; no longer C1.2, RRST.1, U$3./RESET
- net N$31: now also J2.1, Q1.D, R10.1; no longer R18.2, T_HSS.B
- net N$6: now also J2.6, J5.2; no longer J5.1, X1G$1.2
- net RST: now also RRST.1, U$3./RESET; no longer C1.1
- net VCC: now also C10.2, C9.2, L1.1, R5.1, R7.2; no longer S2.P
Other:
- note added: "(optional) Resistor may cause trouble"
- note removed: "KAMERA_SLEEP PIN"
- note removed: "OPTOKOPPLER"
- note removed: "changed pull up resistor from 1k to 10k."
- moved on the sheet: ICSP, J5, VD5, VD6

Commit message: controller6: minor layout changes
Parts:
- C4, C5: device SparkFun-Passives:CAP1206 -> SparkFun-Passives:CAP0805
- RRST: device SparkFun-Passives:RESISTOR1206 -> SparkFun-Passives:RESISTOR0805-RES
Connections:
- removed net BTN_D: U$3.PF6(ADC6/TDO)
- removed net BTN_L: U$3.PF1(ADC1)
- removed net BTN_R: U$3.PF5(ADC5/TMS)
- removed net BTN_U: U$3.PF4(ADC4/TCK)
- new net FOO1: U$3.PB5(OC1A/ADC12/!OC4B)
- new net FOO2: U$3.PB6(OC1B/OC4B/ADC13)
- net BTN: now also U$3.PF7(ADC7(TDI); no longer U$3.PF0(ADC0)
- net CAM1: now also U$3.PF1(ADC1); no longer U$3.PB6(OC1B/OC4B/ADC13)
- net CAM2: now also U$3.PF4(ADC4/TCK); no longer U$3.PC6(OC3A/!OC4A)
- net CAM3: now also U$3.PF5(ADC5/TMS)
- net CAM4: now also U$3.PF6(ADC6/TDO)
- net CAM_EN: now also U$3.PC6(OC3A/!OC4A); no longer U$3.PF7(ADC7(TDI)
- net GND: now also S1.2; no longer S1.1
- net VD_DIRECT: now also U$3.PF0(ADC0); no longer U$3.PB5(OC1A/ADC12/!OC4B)
Changed lines of the file:
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@@
 <part name="GND22" library="SparkFun-Aesthetics" deviceset="GND" device=""/>
 <part name="ICSP" library="SparkFun-Connectors" deviceset="M03X2" device="FEMALE"/>
-<part name="RRST" library="SparkFun-Passives" deviceset="RESISTOR" device="1206"/>
+<part name="RRST" library="SparkFun-Passives" deviceset="RESISTOR" device="0805-RES"/>
 <part name="RUSB1" library="SparkFun-Passives" deviceset="RESISTOR" device="0805-RES"/>
 <part name="RUSB2" library="SparkFun-Passives" deviceset="RESISTOR" device="0805-RES"/>
@@
 <part name="GND14" library="SparkFun-Aesthetics" deviceset="GND" device=""/>
 <part name="U$3" library="adafruit" deviceset="ATMEGA32U4" device="-AU" value=""/>
-<part name="C4" library="SparkFun-Passives" deviceset="CAP" device="1206" value="22pF"/>
-<part name="C5" library="SparkFun-Passives" deviceset="CAP" device="1206" value="22pF"/>
+<part name="C4" library="SparkFun-Passives" deviceset="CAP" device="0805" value="22pF"/>
+<part name="C5" library="SparkFun-Passives" deviceset="CAP" device="0805" value="22pF"/>
 <part name="GND19" library="SparkFun-Aesthetics" deviceset="GND" device=""/>
 <part name="GND20" library="SparkFun-Aesthetics" deviceset="GND" device=""/>
@@
 <instance part="S1" gate="S" x="53.34" y="22.86"/>
 <instance part="R5" gate="G$1" x="66.04" y="27.94" rot="R270"/>
-<instance part="GND27" gate="1" x="40.64" y="22.86" rot="R270"/>
+<instance part="GND27" gate="1" x="40.64" y="20.32" rot="R270"/>
 <instance part="SUPPLY5" gate="G$1" x="66.04" y="35.56"/>
 <instance part="Q1" gate="G$1" x="198.12" y="154.94"/>
@@
 <pinref part="GND18" gate="1" pin="GND"/>
 <wire x1="185.42" y1="48.26" x2="187.96" y2="48.26" width="0.1524" layer="91"/>
-</segment>
-<segment>
-<pinref part="GND27" gate="1" pin="GND"/>
-<pinref part="S1" gate="S" pin="1"/>
-<wire x1="43.18" y1="22.86" x2="48.26" y2="22.86" width="0.1524" layer="91"/>
 </segment>
 <segment>
@@
 <pinref part="R14" gate="G$1" pin="1"/>
 </segment>
+<segment>
+<pinref part="GND27" gate="1" pin="GND"/>
+<pinref part="S1" gate="S" pin="2"/>
+<wire x1="43.18" y1="20.32" x2="48.26" y2="20.32" width="0.1524" layer="91"/>
+</segment>
 </net>
 <net name="CAM_OUT" class="2">
@@
 </net>
 <net name="CAM1" class="0">
-<segment>
-<pinref part="U$3" gate="G$1" pin="PB6(OC1B/OC4B/ADC13)"/>
-<wire x1="132.08" y1="121.92" x2="154.94" y2="121.92" width="0.1524" layer="91"/>
-<label x="154.94" y="121.92" size="1.778" layer="95"/>
-</segment>
 <segment>
 <pinref part="Q1" gate="G$1" pin="G"/>
@@
 <label x="180.34" y="154.94" size="1.778" layer="95" rot="R90"/>
 </segment>
+<segment>
+<pinref part="U$3" gate="G$1" pin="PF1(ADC1)"/>
+<wire x1="132.08" y1="154.94" x2="154.94" y2="154.94" width="0.1524" layer="91"/>
+<label x="154.94" y="154.94" size="1.778" layer="95"/>
+</segment>
 </net>
 <net name="CAM2" class="0">
-<segment>
-<pinref part="U$3" gate="G$1" pin="PC6(OC3A/!OC4A)"/>
-<wire x1="132.08" y1="132.08" x2="154.94" y2="132.08" width="0.1524" layer="91"/>
-<label x="154.94" y="132.08" size="1.778" layer="95"/>
-</segment>
 <segment>
 <pinref part="Q2" gate="G$1" pin="G"/>
@@
 <label x="180.34" y="137.16" size="1.778" layer="95" rot="R90"/>
 </segment>
+<segment>
+<pinref part="U$3" gate="G$1" pin="PF4(ADC4/TCK)"/>
+<wire x1="132.08" y1="152.4" x2="154.94" y2="152.4" width="0.1524" layer="91"/>
+<label x="154.94" y="152.4" size="1.778" layer="95"/>
+</segment>
 </net>
 <net name="BATT_VCC" class="2">
@@
 <label x="50.8" y="165.1" size="1.778" layer="95" rot="R90"/>
 <pinref part="S2" gate="1" pin="O"/>
-</segment>
-</net>
-<net name="CAM_EN" class="0">
-<segment>
-<pinref part="U$3" gate="G$1" pin="PF7(ADC7(TDI)"/>
-<wire x1="132.08" y1="144.78" x2="154.94" y2="144.78" width="0.1524" layer="91"/>
-<label x="154.94" y="144.78" size="1.778" layer="95"/>
 </segment>
 </net>
@@
 <net name="VD_DIRECT" class="0">
 <segment>
-<pinref part="U$3" gate="G$1" pin="PB5(OC1A/ADC12/!OC4B)"/>
-<wire x1="132.08" y1="119.38" x2="154.94" y2="119.38" width="0.1524" layer="91"/>
-<label x="154.94" y="119.38" size="1.778" layer="95"/>
+<pinref part="U$3" gate="G$1" pin="PF0(ADC0)"/>
+<wire x1="132.08" y1="157.48" x2="154.94" y2="157.48" width="0.1524" layer="91"/>
+<label x="154.94" y="157.48" size="1.778" layer="95"/>
 </segment>
 </net>
@@
 </segment>
 </net>
-<net name="BTN_D" class="0">
-<segment>
-<pinref part="U$3" gate="G$1" pin="PF6(ADC6/TDO)"/>
-<wire x1="132.08" y1="147.32" x2="154.94" y2="147.32" width="0.1524" layer="91"/>
-<label x="154.94" y="147.32" size="1.778" layer="95"/>
-</segment>
-</net>
-<net name="BTN_L" class="0">
-<segment>
-<pinref part="U$3" gate="G$1" pin="PF1(ADC1)"/>
-<wire x1="132.08" y1="154.94" x2="154.94" y2="154.94" width="0.1524" layer="91"/>
-<label x="154.94" y="154.94" size="1.778" layer="95"/>
-</segment>
-</net>
-<net name="BTN_R" class="0">
-<segment>
-<pinref part="U$3" gate="G$1" pin="PF5(ADC5/TMS)"/>
-<wire x1="132.08" y1="149.86" x2="154.94" y2="149.86" width="0.1524" layer="91"/>
-<label x="154.94" y="149.86" size="1.778" layer="95"/>
-</segment>
-</net>
-<net name="BTN_U" class="0">
-<segment>
-<pinref part="U$3" gate="G$1" pin="PF4(ADC4/TCK)"/>
-<wire x1="132.08" y1="152.4" x2="154.94" y2="152.4" width="0.1524" layer="91"/>
-<label x="154.94" y="152.4" size="1.778" layer="95"/>
-</segment>
-</net>
 <net name="N$10" class="0">
 <segment>
@@
 </segment>
 <segment>
-<pinref part="U$3" gate="G$1" pin="PF0(ADC0)"/>
-<wire x1="132.08" y1="157.48" x2="154.94" y2="157.48" width="0.1524" layer="91"/>
-<label x="154.94" y="157.48" size="1.778" layer="95"/>
+<pinref part="U$3" gate="G$1" pin="PF7(ADC7(TDI)"/>
+<wire x1="132.08" y1="144.78" x2="154.94" y2="144.78" width="0.1524" layer="91"/>
+<label x="154.94" y="144.78" size="1.778" layer="95"/>
 </segment>
 </net>
@@
 <label x="180.34" y="119.38" size="1.778" layer="95" rot="R90"/>
 </segment>
+<segment>
+<pinref part="U$3" gate="G$1" pin="PF5(ADC5/TMS)"/>
+<wire x1="132.08" y1="149.86" x2="154.94" y2="149.86" width="0.1524" layer="91"/>
+<label x="154.94" y="149.86" size="1.778" layer="95"/>
+</segment>
 </net>
 <net name="CAM4" class="0">
@@
 <junction x="238.76" y="175.26"/>
 <label x="218.44" y="175.26" size="1.778" layer="95"/>
+</segment>
+<segment>
+<pinref part="U$3" gate="G$1" pin="PF6(ADC6/TDO)"/>
+<wire x1="132.08" y1="147.32" x2="154.94" y2="147.32" width="0.1524" layer="91"/>
+<label x="154.94" y="147.32" size="1.778" layer="95"/>
 </segment>
 </net>
@@
 </segment>
 </net>
+<net name="FOO1" class="0">
+<segment>
+<pinref part="U$3" gate="G$1" pin="PB5(OC1A/ADC12/!OC4B)"/>
+<wire x1="132.08" y1="119.38" x2="154.94" y2="119.38" width="0.1524" layer="91"/>
+<label x="154.94" y="119.38" size="1.778" layer="95"/>
+</segment>
+</net>
+<net name="CAM_EN" class="0">
+<segment>
+<pinref part="U$3" gate="G$1" pin="PC6(OC3A/!OC4A)"/>
+<wire x1="132.08" y1="132.08" x2="154.94" y2="132.08" width="0.1524" layer="91"/>
+<label x="154.94" y="132.08" size="1.778" layer="95"/>
+</segment>
+</net>
+<net name="FOO2" class="0">
+<segment>
+<pinref part="U$3" gate="G$1" pin="PB6(OC1B/OC4B/ADC13)"/>
+<wire x1="132.08" y1="121.92" x2="154.94" y2="121.92" width="0.1524" layer="91"/>
+<label x="154.94" y="121.92" size="1.778" layer="95"/>
+</segment>
+</net>
