File: eagle/controller8/controller8.brd (EAGLE design)
At the start: 30 x 65 mm, 88 parts, among them IC1 ILD213T, IC2 ILD213T, Q1 2.5A/30V, Q2 200mA/50V, U2 MP2307, U3 MP2307, X1 1501_04, X2 ZX62D-B-5PA8

Commit message: controller 7/8/9
Parts:
- removed C1: 0.1uF (low leakage), SparkFun-Capacitors:1206
- removed C10, C16, C17, C9: 22uF / 6.3V, SparkFun-Capacitors:1206
- removed C11, C12, C18, C19: 10uF / 25V, SparkFun-Capacitors:1206
- removed C13, C6: 10nF, SparkFun-Capacitors:1206
- removed C14, C7: 3.9nF, SparkFun-Capacitors:0805
- removed C15, C8: 0.1uF, SparkFun-Capacitors:0805
- removed C2: 1uF, SparkFun-Capacitors:1206
- removed C3: 10uF, SparkFun-Passives:1206
- removed C4, C5: 22pF, SparkFun-Passives:0805
- removed F2: PTCSMD-W, SparkFun-PowerIC:PTC-1206-WIDE
- removed ICSP1: (no value), SparkFun-Connectors:2X3
- removed L1, L2: 10uH / 4A, SparkFun-Passives:SRU1038
- removed R1, R4: 6.8k, SparkFun-Resistors:0805
- removed R2, R6: 10k / 1%, SparkFun-Resistors:0805
- removed R22, RRST, RUSB1, RUSB2: (no value), SparkFun-Passives:1206
- removed R23, R24: 100K, SparkFun-Resistors:0805
- removed R3: 44k / 1%, SparkFun-Resistors:0805
- removed R7: 26.1k / 1%, SparkFun-Resistors:0805
- removed RTC2: DS3231M, SparkFun-DigitalIC:SOIC8
- removed RV1: (no value), SparkFun-Electromechanical:ALPS_POT
- removed U$3: (no value), adafruit:TQFP44
- removed U$8: PIZERO_12PIN, pizero:PIZERO_12PIN
- removed U2, U3: MP2307, SparkFun-AnalogIC:SO08
- removed X2: ZX62D-B-5PA8, zx62d-b-5pa8-oshpark_10:ZX62D-B-5PA8
- removed Y1: (no value), SparkFun-FreqCtrl:CRYSTAL-SMD-5X3
- added J11, J8: (no value), SparkFun-Connectors:1X14_LOCK
- added J12, J14, J15: (no value), SparkFun-Connectors:1X05_LOCK
- added J13: (no value), SparkFun-Connectors:AVR_ICSP
- U$1: value PIZERO_12PIN -> PIZERO_THROUGH_HOLE; device pizero:PIZERO_12PIN -> pizero:PIZERO_THOUGH_HOLE
- moved S1 66.0 mm to (10.8, 3.56)
- moved D2 66.0 mm to (19.1, 3.81)
- moved J5 54.1 mm to (3.30, 41.5), turned to 90 degrees
- moved R_LED 52.1 mm to (19.1, 10.2), turned to 0 degrees
- moved R5 51.7 mm to (19.1, 7.62), turned to 180 degrees
- moved R10 44.5 mm to (15.2, 34.9)
- moved Q1 43.3 mm to (15.2, 38.1)
- moved R19 39.0 mm to (15.9, 23.5), turned to 0 degrees
- moved R18 37.9 mm to (15.9, 21.6), turned to 0 degrees
- moved Q2 37.4 mm to (19.1, 37.5)
- moved S4 35.1 mm to (73.7, 52.8), turned to 180 degrees
- moved IC1 33.0 mm to (15.9, 29.2)
- moved IC2 33.0 mm to (21.6, 29.2)
- moved JP1 33.0 mm to (22.2, 35.6)
- moved J2 32.4 mm to (26.3, 49.0)
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Connections:
- removed net ANALOG_IO: U$1.24, U$3.30
- removed net BUCK_EN: U$1.16, U$3.1
- removed net CAM_EN1: U$1.20, U$3.37
- removed net CAM_EN2: U$1.15, U$3.40
- removed net DB_ANALOG_IO: RV1.P$2, U$8.24
- removed net FOOA: U$3.28
- removed net MISO: ICSP1.1, U$3.11
- removed net MOSI: ICSP1.4, U$3.10
- removed net N$10: RUSB1.2, X2.2
- removed net N$11: RUSB2.2, X2.3
- removed net N$14: C8.2, U2.8
- removed net N$17: C6.2, L1.2, U2.3
- removed net N$2: R23.2, U2.7
- removed net N$20: C2.2, U$3.6
- removed net N$21: C7.1, R4.1
- removed net N$22: C3.1, F2.2, U$3.7
- removed net N$23: C7.2, U2.6
- removed net N$24: R6.1, R7.1, U2.5
- removed net N$25: C15.2, U3.8
- removed net N$26: C13.2, L2.2, U3.3
- removed net N$27: C13.1, U3.1
- removed net N$28: C14.1, R1.1
- removed net N$29: C14.2, U3.6
- removed net N$3: C6.1, U2.1
- removed net N$30: R2.1, R3.1, U3.5
- removed net N$38: F2.1, X2.1
- removed net N$4: RUSB1.1, U$3.3
- removed net N$43: R22.2, RV1.P$1
- removed net N$5: RUSB2.1, U$3.4
- removed net N$8: C4.2, U$3.17, Y1.3
- removed net N$9: C5.2, U$3.16, Y1.1
- removed net NC: U$1.11
- removed net NC_2: U$2.11
- removed net PB_BUCK_EN: R24.2, U$2.16, U3.7
- removed net PB_CONV_5V: C16.2, C17.2, L2.1, R3.2, U$2.2
- removed net PROFET1: U$1.18, U$3.39
- removed net PROFET2: U$1.19, U$3.36
- removed net PROFET3: U$1.17, U$3.38
- removed net RST: ICSP1.5, RRST.1, U$3.13
- removed net RX: U$1.8, U$3.20
- removed net SCK: ICSP1.3, U$3.9
- removed net TX: U$1.10, U$3.21
- removed net VCC-ISO: C10.2, C9.2, L1.1, R7.2, U$2.14
- removed net VD_DIRECT: U$1.13, U$3.41
- net 3.3V: no longer RV1.P$3, U$8.6
- net BATT_VCC: no longer C11.1, C12.2, C18.1, C19.2, R23.1, R24.1, U2.2, U3.2
- net BTN: no longer U$1.22, U$3.32
- net CAM1: no longer U$3.29
- net CAM2: no longer U$3.27
- net CAM3: no longer U$3.26
- net CAM4: no longer U$3.25
- net CONV_5V: no longer U$1.2
- net DB_BTN: no longer U$8.22
- net DB_SCL: no longer U$8.21
- net DB_SDA: no longer U$8.23
- net GND: no longer C1.2, C2.1, C3.2, C4.1, C5.1, ICSP1.6, RTC2.5, U$1.6, U$3.15, U$3.23, U$3.33, U$3.35, U$3.43, U$3.5, X2.5
- net GND-ISO: no longer C10.1, C11.2, C12.1, C15.1, C16.1, C17.1, C18.2, C19.1, C8.1, C9.1, R1.2, R2.2, R4.2, R6.2, U$2.6, U2.4, U2.BTM, U2.P$1, U3.4, U3.BTM, U3.P$1
- net LED: no longer U$3.31
- net N$39: no longer C1.1, RTC2.6
- net PB_CAM_EN1: no longer U$2.20
- net PB_CAM_EN2: no longer U$2.15
- net PB_PROFET_1: no longer U$2.18
- net PB_PROFET_2: no longer U$2.19
- net PB_PROFET_3: no longer U$2.17
- net PB_VD_DIRECT: no longer U$2.13
- net SCL: no longer RTC2.8, U$1.21, U$3.18
- net SDA: no longer RTC2.7, U$1.23, U$3.19
- net SWITCH_USB_VCC: no longer U$3.22
- net VCC: no longer ICSP1.2, RRST.2, RTC2.2, U$1.14, U$3.14, U$3.2, U$3.24, U$3.34, U$3.42, U$3.44
- net VCC_2: no longer R22.1, U$8.14
Routing:
- net GND-ISO: track 172.2 -> 0.00 mm, vias 1 -> 0
- net GND: track 165.4 -> 0.00 mm, vias 3 -> 0
- net VCC: track 148.7 -> 0.00 mm, vias 5 -> 0
- net BATT_VCC: track 101.7 -> 0.00 mm, vias 1 -> 0
- net 3.3V: track 85.3 -> 0.00 mm
- net CONV_5V: track 54.8 -> 0.00 mm, vias 1 -> 0
- net SDA: track 46.3 -> 0.00 mm, vias 2 -> 0
- net BTN: track 46.1 -> 0.00 mm
- net N$34: track 44.6 -> 0.00 mm
- net SCL: track 42.7 -> 0.00 mm, vias 2 -> 0
- net GNDA: track 42.1 -> 0.00 mm
- net VCC_2: track 41.1 -> 0.00 mm
- net DB_SCL: track 33.5 -> 0.00 mm
- net PB_BUCK_EN: track 33.4 -> 0.00 mm, vias 1 -> 0
- net LED: track 32.5 -> 0.00 mm, vias 2 -> 0
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Other:
- board text removed: "7"
- board text removed: "BOARD1"
- board text removed: "BOX"
- board text removed: "CONTROLLER7"
- board text removed: "POWERBOARD1"
- board text removed: "RTC"
- board text removed: "TIME"
