File: eagle/controller9/controller9.sch (EAGLE design)
At the start: 34 parts, among them IC1 ILD213T, IC2 ILD213T, Q1 2.5A/30V, Q2 200mA/50V, Q3 FDD4141TO252, X1 1501_04

Commit message: controller10
Parts:
- removed J13: (no value), SparkFun-Connectors:M05X2PTH
- removed Q1: 2.5A/30V, SparkFun-DiscreteSemi:MOSFET-PCHANNELDMG2307L
- removed Q2: 200mA/50V, SparkFun-DiscreteSemi:MOSFET-NCHANNELBSS138
- removed R10: (no value), SparkFun-Passives:RESISTOR0805-RES
- removed SH1: SHORT-HT5, shorts-old:SHORT-HT5
- removed TP1, TP2, TP3: TEST-POINT3X5, SparkFun-Passives:TEST-POINT3X5
- removed T_HSS: (no value), SparkFun-DiscreteSemi:TRANSISTOR_NPN2N3904
- added H1: MOUNT-HOLE3.2, holes:MOUNT-HOLE3.2
- added J1: (no value), SparkFun-Connectors:M05X2PTH
- added Q4: 200mA/50V, SparkFun-DiscreteSemi:MOSFET-NCHANNELBSS138
- J2: device SparkFun-Connectors:M04X2 -> SparkFun-Connectors:M03X2FEMALE
- R13, VD1, VD2: device SparkFun-Passives:RESISTOR1206 -> SparkFun-Passives:RESISTOR0805-RES
- R_LED: device SparkFun-Resistors:RESISTOR1206 -> SparkFun-Resistors:RESISTOR0805-RES
Connections:
- removed net CAM_EN1: J8.19
- removed net CAM_OUT1: J9.2
- removed net GND-ISO: SH1.P$1, VD2.1
- removed net GNDA: J7.1, J9.1, SH1.P$2
- removed net N$1: J2.4, TP2.1
- removed net N$34: IC1.ET1, IC1.ET2, IC2.ET1, IC2.ET2, J2.7, JP1.2, X1.1
- removed net N$35: J2.8, Q1.D
- removed net N$36: Q1.G, Q2.S, R10.1
- removed net N$6: J2.6, TP1.1
- removed net PB_VD_DIRECT: VD1.1, VD2.2
- removed net SWITCH_USB_VCC: Q2.G
- new net N$4: IC1.ET1, IC1.ET2, IC2.ET1, IC2.ET2, J2.6, X1.1
- new net RX: J1.8, J8.2
- new net SCL: J8.6
- new net SDA: J8.7
- new net TX: J1.10, J8.3
- net BTN: now also J8.18; no longer J8.8
- net BUCK_EN: now also J8.12
- net CAM1: now also J8.16; no longer J8.15
- net CAM2: now also J8.15; no longer J8.14
- net CAM3: now also J8.14; no longer J8.13
- net CAM4: now also J8.13
- net CAM_EN: now also J8.21
- net CAM_OUT: now also J9.2
- net CONV_5V: now also J1.2; no longer Q1.S, R10.2
- net GND: now also J1.6, J7.1, J9.1, Q4.D, VD2.1; no longer Q2.D, TP3.1, T_HSS.E
- net LED: now also J8.19
- net N$16: now also JP1.2
- net N$2: now also Q4.G; no longer T_HSS.B
- net N$3: now also Q4.S; no longer T_HSS.C
- net VD_DIRECT: now also J8.20, VD1.1, VD2.2; no longer J8.18
Other:
- note removed: "5V über mosfet"
- moved on the sheet: JP1, R1, R13
