File: eagle/controller10/controller10.brd (EAGLE design)
At the start: 36.8 x 64.8 mm, 63 parts, among them IC1 ILD213T, IC2 ILD213T, J2 FEMALE 2x3, Q2 200mA/50V, Q4 200mA/50V, Q5 200mA/50V, U3 MP2307, X1 1501_04, X2 ZX62D-B-5PA8

Commit message: controller10: version sent to fab
Parts:
- removed U$1: PIZERO_THROUGH_HOLE, pizero:PIZERO_THOUGH_HOLE
- H1, H2: value MOUNT-HOLE3.3 -> MOUNT-HOLE2.8; device holes:3,3 -> holes:2,8
- R12: value 10k -> 20k
- moved R9 0.13 mm to (12.6, 55.2)
Routing:
- net ZERO_5V: track 19.1 -> 24.5 mm
- net GND: track 126.7 -> 129.4 mm, vias 2 -> 3
- net VCC: track 105.0 -> 105.5 mm

Commit message: update
Parts:
- moved R24 1.27 mm to (8.89, 55.2), turned to 270 degrees
Routing:
- net PB_BUCK_EN: track 10.7 -> 11.7 mm
- net N$1: track 14.1 -> 13.2 mm
Changed lines of the file:
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@@
 <?xml version="1.0" encoding="utf-8"?>
 <!DOCTYPE eagle SYSTEM "eagle.dtd">
-<eagle version="8.2.0">
+<eagle version="8.2.1">
 <drawing>
 <settings>
@@
 <attribute name="OC_NEWARK" value="unknown" x="38.1" y="55.88" size="1.778" layer="27" rot="R270" display="off"/>
 </element>
-<element name="R24" library="SparkFun-Resistors" package="0805" value="100K" x="8.89" y="53.975" smashed="yes"/>
+<element name="R24" library="SparkFun-Resistors" package="0805" value="100K" x="8.89" y="55.245" smashed="yes" rot="R270"/>
 <element name="F2" library="SparkFun-PowerIC" package="PTC-1206-WIDE" value="PTCSMD-W" x="10.033" y="8.001" smashed="yes" rot="R180"/>
 <element name="J1" library="SparkFun-Connectors" package="AVR_ICSP" value="" x="32.385" y="13.462" smashed="yes">
@@
 <wire x1="2.667" y1="49.911" x2="1.651" y2="48.895" width="0.6604" layer="1"/>
 <wire x1="2.667" y1="49.911" x2="2.845" y2="50.165" width="0.6604" layer="1"/>
-<wire x1="8.763" y1="54.737" x2="8.001" y2="53.975" width="0.6604" layer="1"/>
-<wire x1="8.763" y1="54.864" x2="8.763" y2="54.737" width="0.6604" layer="1"/>
-<wire x1="9.144" y1="55.245" x2="8.763" y2="54.864" width="0.6604" layer="1"/>
-<wire x1="11.673" y1="55.245" x2="9.144" y2="55.245" width="0.6604" layer="1"/>
-<wire x1="8.001" y1="53.975" x2="7.99" y2="53.975" width="0.6604" layer="1"/>
-<wire x1="14.351" y1="54.102" x2="14.351" y2="53.086" width="0.6604" layer="1"/>
-<wire x1="16.383" y1="55.499" x2="14.351" y2="54.102" width="0.6604" layer="1"/>
-<wire x1="16.383" y1="59.055" x2="16.383" y2="55.499" width="0.6604" layer="1"/>
-<wire x1="13.843" y1="61.595" x2="14.6685" y2="60.7695" width="0.6604" layer="1"/>
-<wire x1="14.6685" y1="60.7695" x2="16.383" y2="59.055" width="0.6604" layer="1"/>
-<wire x1="14.351" y1="53.086" x2="14.25" y2="52.965" width="0.6604" layer="1"/>
+<wire x1="10.541" y1="56.134" x2="8.763" y2="56.134" width="0.6604" layer="1"/>
+<wire x1="11.673" y1="55.245" x2="10.541" y2="56.134" width="0.6604" layer="1"/>
+<wire x1="14.605" y1="54.102" x2="14.605" y2="53.086" width="1.016" layer="1"/>
+<wire x1="16.383" y1="55.499" x2="14.605" y2="54.102" width="1.016" layer="1"/>
+<wire x1="16.383" y1="59.055" x2="16.383" y2="55.499" width="1.016" layer="1"/>
+<wire x1="13.843" y1="61.595" x2="14.0335" y2="61.4045" width="1.016" layer="1"/>
+<wire x1="14.0335" y1="61.4045" x2="16.383" y2="59.055" width="1.016" layer="1"/>
+<wire x1="14.605" y1="53.086" x2="14.25" y2="52.965" width="0.6604" layer="1"/>
 <wire x1="13.843" y1="61.595" x2="13.7922" y2="61.595" width="0.6604" layer="1"/>
 <wire x1="13.843" y1="61.595" x2="13.843" y2="57.785" width="0.6604" layer="16"/>
 <wire x1="13.843" y1="57.785" x2="13.84" y2="57.785" width="0.6604" layer="16"/>
 <wire x1="13.843" y1="61.595" x2="13.7922" y2="61.595" width="0.6604" layer="16"/>
-<wire x1="14.6685" y1="60.7695" x2="11.684" y2="57.404" width="0.6604" layer="1"/>
-<wire x1="11.684" y1="57.404" x2="11.673" y2="55.245" width="0.6604" layer="1"/>
-<wire x1="3.683" y1="54.102" x2="3.175" y2="54.102" width="0.6604" layer="1"/>
-<wire x1="5.207" y1="55.626" x2="3.683" y2="54.102" width="0.6604" layer="1"/>
-<wire x1="6.985" y1="55.626" x2="5.207" y2="55.626" width="0.6604" layer="1"/>
-<wire x1="8.128" y1="54.483" x2="6.985" y2="55.626" width="0.6604" layer="1"/>
+<wire x1="14.0335" y1="61.4045" x2="11.684" y2="58.674" width="0.6604" layer="1"/>
+<wire x1="11.684" y1="58.674" x2="11.673" y2="55.245" width="0.6604" layer="1"/>
+<wire x1="3.048" y1="54.102" x2="3.175" y2="54.102" width="0.6604" layer="1"/>
+<wire x1="5.08" y1="56.134" x2="3.048" y2="54.102" width="0.6604" layer="1"/>
+<wire x1="7.112" y1="56.134" x2="5.08" y2="56.134" width="0.6604" layer="1"/>
 <wire x1="3.175" y1="54.102" x2="2.845" y2="53.975" width="0.6604" layer="1"/>
-<wire x1="8.128" y1="54.483" x2="7.99" y2="53.975" width="0.6604" layer="1"/>
+<wire x1="7.112" y1="56.134" x2="8.89" y2="56.145" width="0.6604" layer="1"/>
+<wire x1="8.89" y1="56.145" x2="8.763" y2="56.134" width="0" layer="19" extent="1-1"/>
 </signal>
 <signal name="N$4">
@@
 <wire x1="11.557" y1="45.72" x2="12.7" y2="46.863" width="0.254" layer="1"/>
 <wire x1="10.8712" y1="45.72" x2="11.557" y2="45.72" width="0.254" layer="1"/>
-<wire x1="9.906" y1="53.975" x2="9.79" y2="53.975" width="0.254" layer="1"/>
+<wire x1="9.906" y1="53.975" x2="8.89" y2="54.345" width="0.254" layer="1"/>
 </signal>
 <signal name="N$12">
@@
 <wire x1="12.954" y1="51.562" x2="15.621" y2="48.895" width="0.254" layer="1"/>
 <wire x1="12.954" y1="54.864" x2="12.954" y2="51.562" width="0.254" layer="1"/>
-<wire x1="12.954" y1="54.864" x2="13.716" y2="55.245" width="0.254" layer="1"/>
-<wire x1="14.859" y1="56.134" x2="14.859" y2="57.404" width="0.254" layer="1"/>
-<wire x1="13.716" y1="55.245" x2="14.859" y2="56.134" width="0.254" layer="1"/>
-<wire x1="14.859" y1="57.404" x2="14.25" y2="57.525" width="0.254" layer="1"/>
-<wire x1="13.716" y1="55.245" x2="13.473" y2="55.245" width="0.254" layer="1"/>
+<wire x1="12.954" y1="54.864" x2="13.589" y2="55.372" width="0.254" layer="1"/>
+<wire x1="13.589" y1="57.023" x2="14.224" y2="57.531" width="0.254" layer="1"/>
+<wire x1="13.589" y1="55.372" x2="13.589" y2="57.023" width="0.254" layer="1"/>
+<wire x1="14.224" y1="57.531" x2="14.25" y2="57.525" width="0.254" layer="1"/>
+<wire x1="13.589" y1="55.372" x2="13.473" y2="55.245" width="0.254" layer="1"/>
 </signal>
 <signal name="N$6">
@@
 <contactref element="Q1" pad="3"/>
 <contactref element="J9" pad="2"/>
-<wire x1="27.686" y1="60.706" x2="27.686" y2="61.595" width="0.6604" layer="1"/>
-<wire x1="22.225" y1="55.245" x2="27.686" y2="60.706" width="0.6604" layer="1"/>
+<wire x1="27.686" y1="60.706" x2="27.686" y2="61.595" width="1.016" layer="1"/>
+<wire x1="22.225" y1="55.245" x2="27.686" y2="60.706" width="1.016" layer="1"/>
 <wire x1="27.686" y1="61.595" x2="27.7622" y2="61.595" width="0.6604" layer="1"/>
 <wire x1="22.225" y1="55.245" x2="21.55" y2="55.245" width="0.6604" layer="1"/>
