File: eagle/controller10/controller10.sch (EAGLE design)
At the start: 59 parts, among them IC1 ILD213T, IC2 ILD213T, J2 FEMALE 2x3, Q3 FDD4141TO252, Q4 200mA/50V, U3 MP2307, X1 1501_04, X2 ZX62D-B-5PA8

Commit message: controller10 ready for fab
Parts:
- removed ICSP1: (no value), SparkFun-Connectors:M03X2FEMALE
- removed J10: (no value), SparkFun-Connectors:M02LOCK
- removed PT1: 2PT_GND_TIE, SparkFun-Passives:2PT_GND_TIE
- removed R17: (no value), SparkFun-Passives:RESISTOR1206
- removed S3: (no value), SparkFun-Electromechanical:SWITCH-SPDTPTH_LOCK
- removed U$7: BTS7008-2EPA, SparkFun-DigitalIC:BTS7008-2EPA
- added J3: (no value), SparkFun-Connectors:M04X2
- added Q1: FDD4141TO252, transistor-fet:FDD4141TO252
- added Q2, Q5: 200mA/50V, SparkFun-DiscreteSemi:MOSFET-NCHANNELBSS138
- added R10: 1k, SparkFun-Resistors:RESISTOR0805-RES
- added R14: (no value), SparkFun-Passives:RESISTOR0805-RES
- added R7, R8, R9: 10k, SparkFun-Resistors:RESISTOR0805-RES
- added SH1: SHORT-HT5, shorts:SHORT-HT5
- R11, R12: value (none) -> 10k; device SparkFun-Passives:RESISTOR1206 -> SparkFun-Resistors:RESISTOR0805-RES
- R13, R16: device SparkFun-Passives:RESISTOR1206 -> SparkFun-Passives:RESISTOR0805-RES
Connections:
- removed net BATT_VCC_RAW: J7.2, S3.O
- removed net CAM_EN1: R11.1, U$3.PF6(ADC6/TDO), U$7.IN0
- removed net CAM_EN2: R12.2, U$3.PF1(ADC1), U$7.IN1
- removed net CAM_OUT1: J9.2, U$7.OUT0
- removed net CAM_OUT2: J10.2, U$7.OUT1
- removed net FOOA: U$3.PB4(ADC11)
- removed net GND-ISO: R12.1, U$7.GND
- removed net PROFET1: R17.1, U$3.PF4(ADC4/TCK), U$7.DEN
- removed net PROFET2: U$3.PF7(ADC7(TDI), U$7.IS
- removed net PROFET3: R16.2, U$3.PF5(ADC5/TMS), U$7.DSEL
- removed net SWITCH_USB_VCC: U$3.PD5(XCK/CTS)
- new net CAM_EN: R10.1, U$3.PC6(OC3A/!OC4A)
- new net CAM_OUT: J9.2, Q1.D
- new net FOO1: U$3.PF5(ADC5/TMS)
- new net FOO2: U$3.PF0(ADC0)
- new net FOO3: U$3.PB0(SS)
- new net FOO4: U$3.PF6(ADC6/TDO)
- new net FOO5: U$3.PC7(ICP3/CLK0/OC4A)
- new net FOO6: U$3.PB5(OC1A/ADC12/!OC4B)
- new net FOO7: U$3.PF7(ADC7(TDI)
- new net FOO8: U$3.PF4(ADC4/TCK)
- new net N$1: Q1.G, Q2.D, R9.2
- new net N$6: Q2.G, R10.2
- new net SCL: J3.2, R16.2, U$3.PD0(INT0/OC0B/SCL)
- new net SDA: J3.1, R14.1, U$3.PD1(INT1/SDA)
- new net ZERO_3.3V: J1.10, Q5.G, R7.1
- new net ZERO_RX: J1.1, R11.2, R12.1
- new net ZERO_TX: J1.3, Q5.S, R7.2
- net BATT_VCC: now also J7.2, Q1.S, R9.1; no longer S3.P, U$7.VS
- net BTN: now also U$3.PF1(ADC1); no longer U$3.PC7(ICP3/CLK0/OC4A)
- net CAM1: now also U$3.PB4(ADC11); no longer U$3.PB5(OC1A/ADC12/!OC4B)
- net CONV_5V: now also SH1.P$1; no longer PT1.P$1
- net GND: now also J3.8, Q2.S, Q4.S, R12.2; no longer ICSP1.6, J10.1, Q4.D, R11.2, R16.1, R17.2
- net LED: now also U$3.PE6(INT.6/AIN0); no longer U$3.PC6(OC3A/!OC4A)
- net MISO: now also J3.3; no longer ICSP1.1
- net MOSI: now also J3.6; no longer ICSP1.4
- net N$3: now also Q4.D; no longer Q4.S
- net RST: now also J3.7; no longer ICSP1.5
- net RX: now also Q5.D, R8.2; no longer J1.3
- net SCK: now also J3.5; no longer ICSP1.3
- net TX: now also R11.1; no longer J1.1
- net VCC: now also J3.4, R14.2, R16.1, R8.1, SH1.P$2; no longer ICSP1.2, PT1.P$2
- net VD_DIRECT: now also U$3.PB6(OC1B/OC4B/ADC13); no longer U$3.PF0(ADC0)
- net ZERO_EN: now also U$3.PD5(XCK/CTS); no longer U$3.PE6(INT.6/AIN0)
Other:
- note added: "if inactive: pull up or down?"
- note removed: "BTS7008-2EPA"
- moved on the sheet: H1, H2, Q3, Q4, R11, R12, R4, R6

Commit message: controller10: version sent to fab
Parts:
- removed U$1: PIZERO_THROUGH_HOLE, pizero:PIZERO_THROUGH_HOLE
- H1, H2: value MOUNT-HOLE3.3 -> MOUNT-HOLE2.8; device holes:MOUNT-HOLE3.3 -> holes:MOUNT-HOLE2.8
- R12: value 10k -> 20k
