File: eagle/controller14/controller14.brd (EAGLE design)
At the start: 30 x 65 mm, 48 parts, among them IC1 ILD213T, J2 AVR_SPI_PRG_6PTH, J3 USB_A_SMT_FEMALE, J5 FEMALE 2x3, J6 USB_A_SMT_FEMALE, Q2 200mA/50V, Q4 200mA/50V, Q5 200mA/50V, Q7 200mA/50V, X1 1501_04, X2 ZX62D-B-5PA8

Commit message: controller14: progress
Parts:
- removed J5: FEMALE 2x3, SparkFun-Connectors:2X3
- removed S2: (no value), SparkFun-Electromechanical:SWITCH-SPDT-SMD
- removed X2: ZX62D-B-5PA8, zx62d-b-5pa8-oshpark_10:ZX62D-B-5PA8
- added D1, D3: (no value), SparkFun-LED:LED-1206
- added J7: (no value), SparkFun-Connectors:USB-C-16P
- added J8: 2X6 FEMALE, SparkFun-Connectors:2X6
- added Q8: 200mA/50V, SparkFun-DiscreteSemi:SOT23-3
- added R13, R3: 5.1k, SparkFun-Resistors:0603
- added R14, R16: 1k, SparkFun-Resistors:1206
- added S3, S4, S5: MOMENTARY-SWITCH-SPST-PTH-RIGHT-ANGLE-KIT, SparkFun-Switches:TACTILE_SWITCH_PTH_RIGHT_ANGLE_KIT
- added U1: DS3234, SparkFun-Clocks:SO20-0.3
- moved X1 40.9 mm to (9.65, 66.5), turned to 0 degrees
- moved JP1 32.5 mm to (9.65, 60.5)
- moved R_LED 28.5 mm to (21.3, 61.7), flipped to the top
- moved S1 26.1 mm to (50.7, 16.5), turned to 180 degrees
- moved Q6 25.5 mm to (22.9, 32.5), turned to 90 degrees
- moved J6 25.2 mm to (24.6, 32.5), turned to 180 degrees
- moved D2 23.8 mm to (16.9, 60.7), turned to 90 degrees
- moved J4 19.3 mm to (36.6, 61.5)
- moved R10 17.7 mm to (36.7, 42.0)
- moved IC1 16.1 mm to (8.64, 49.5), turned to 0 degrees
- moved Q2 15.6 mm to (34.7, 46.4)
- moved R1 14.8 mm to (14.2, 53.8), turned to 270 degrees
- moved C2 9.71 mm to (18.3, 26.0)
- moved RRST 9.49 mm to (34.8, 20.6)
- moved Q7 8.89 mm to (14.2, 54.9), turned to 90 degrees
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Connections:
- removed net CONV_5V: S2.1
- removed net FOO5: U$3.36
- removed net N$38: F2.1, X2.1
- removed net VD_INT: U$3.38
- new net CC1: J7.A5, R13.2
- new net CC2: J7.B5, R3.2
- new net D+: J7.A6, J7.B6, RUSB2.2
- new net D-: J7.A7, J7.B7, RUSB1.2
- new net DUMMY_LOAD: R14.1, U$3.36
- net EXT1: no longer J5.1
- net EXT2: no longer J5.2
- net EXT3: no longer J5.4
- net EXT4: no longer J5.6
- net GND: now also J7.GND, J7.GND2, J7.SHLD1, J7.SHLD2, J7.SHLD3, J7.SHLD4, J7.SHLD5, J7.SHLD6, J7.SHLD7, J7.SHLD8, Q8.2, R13.1, R3.1, S3.1, S4.1, S5.1; no longer X2.5
- net N$10: now also Q8.1, R14.2; no longer RUSB1.2, X2.2
- net N$11: now also Q8.3, R16.1; no longer RUSB2.2, X2.3
- net SCL: no longer J5.5
- net SDA: no longer J5.3
- net VBUS: no longer S2.3
- net VCC: now also F2.1, J7.VBUS1, J7.VBUS2, R16.2; no longer S2.2
Routing:
- net VCC: track 124.0 -> 58.2 mm, vias 3 -> 1
- net CONV_5V: track 42.6 -> 0.00 mm, vias 1 -> 0
- net SCK: track 42.6 -> 0.00 mm, vias 2 -> 0
- net RST: track 41.9 -> 0.00 mm, vias 2 -> 0
- net MOSI: track 41.7 -> 0.00 mm, vias 2 -> 0
- net MISO: track 37.0 -> 0.00 mm, vias 2 -> 0
- net EXT4: track 19.2 -> 0.02 mm
- net EXT3: track 18.9 -> 0.00 mm, vias 1 -> 0
- net EXT1: track 15.6 -> 0.00 mm, vias 1 -> 0
- net EXT2: track 15.1 -> 0.00 mm, vias 1 -> 0
- net SCL: track 14.9 -> 0.00 mm
- net LED: track 14.7 -> 0.00 mm
- net BTN: track 14.2 -> 0.00 mm
- net SDA: track 13.4 -> 0.00 mm
- net VD_INT: track 13.0 -> 0.00 mm, vias 1 -> 0
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- removed copper zone on layer 1, net CONV_5V

Commit message: controller14: nearly done
Parts:
- removed C1: 0.1uF, SparkFun-Capacitors:1206
- removed F2: PTCSMD-W, SparkFun-PowerIC:PTC-1206-WIDE
- removed J4: (no value), SparkFun-Connectors:1X02
- removed J8: 2X6 FEMALE, SparkFun-Connectors:2X6
- removed R5: (no value), SparkFun-Passives:1206
- removed RAREF: 5k, SparkFun-Passives:1206
- removed S1: TAC_SWITCHSMD, SparkFun-Retired:TACTILE-PTH
- added J5: (no value), SparkFun-Connectors:2X8
- added R17, R18, R19: 10k, SparkFun-Resistors:1206
- J1: device SparkFun-Connectors:AVR_ICSP -> SparkFun-Connectors:1X02
- R13, R3: value 5.1k -> (none); device SparkFun-Resistors:0603 -> SparkFun-Passives:1206
- moved Q8 27.6 mm to (18.3, 4.06), turned to 270 degrees
- moved J2 27.5 mm to (27.7, 21.8), turned to 180 degrees
- moved R3 26.3 mm to (17.5, 20.1), flipped to the bottom, turned to 180 degrees
- moved R16 26.1 mm to (21.3, 3.56)
- moved R14 25.8 mm to (15.2, 4.06), turned to 270 degrees
- moved Q7 25.0 mm to (16.3, 30.0)
- moved R13 23.2 mm to (21.3, 3.56), flipped to the bottom, turned to 90 degrees
- moved R10 23.0 mm to (13.7, 41.7)
- moved R2 22.9 mm to (13.7, 26.9), turned to 180 degrees
- moved R15 20.0 mm to (9.14, 51.8), turned to 0 degrees
- moved R1 19.4 mm to (16.3, 34.5), flipped to the bottom
- moved Q2 19.0 mm to (15.7, 47.8), turned to 90 degrees
- moved RRST 17.8 mm to (17.3, 23.6), turned to 90 degrees
- moved J1 15.3 mm to (4.80, 28.7), turned to 180 degrees
- moved R_LED 12.6 mm to (13.2, 52.1)
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Connections:
- removed net BATT_VCC: J4.1, Q1.2, Q6.2, R1.1, R9.1
- removed net CAM_EN: U$3.25
- removed net EXT4: U$3.26
- removed net FOO2: U$3.41
- removed net N$18 (its old number): C1.2, RAREF.1, U$3.42
- removed net VBUS: C3.1, F2.2, U$3.7
- new net FOO5: U$3.36
- new net SHIELD: J7.SHLD1, J7.SHLD2, J7.SHLD3, J7.SHLD4, J7.SHLD5, J7.SHLD6, J7.SHLD7, J7.SHLD8
- new net SIDEBUTTON1: J5.13, R17.2, S5.2
- new net SIDEBUTTON2: J5.15, R18.2, S4.2
- new net SIDEBUTTON3: J5.12, R19.1, S3.2
- new net ZERO_3.3V2: J1.1, R17.1, R18.1, R19.2
- net BTN: no longer R5.2, S1.4
- net CAM1: now also U$3.28; no longer U$3.27
- net CAM1_EN: now also U$3.25
- net CAM2: now also U$3.27; no longer U$3.28
- net CAM2_EN: now also U$3.26
- net DUMMY_LOAD: now also U$3.41; no longer U$3.36
- net GND: now also J5.6; no longer C1.1, J1.5, J4.2, J7.SHLD1, J7.SHLD2, J7.SHLD3, J7.SHLD4, J7.SHLD5, J7.SHLD6, J7.SHLD7, J7.SHLD8, S1.2
- net VCC: now also C3.1, Q1.2, Q6.2, R1.1, R9.1, U$3.7; no longer F2.1, R5.1, RAREF.2
- net ZERO_3.3V: now also J5.1; no longer J1.10
- net ZERO_5V: now also J5.2; no longer J1.9
- net ZERO_RX: now also J5.10; no longer J1.1
- net ZERO_TX: now also J5.8; no longer J1.3
Routing:
- net VCC: track 58.2 -> 154.2 mm, vias 1 -> 3
- net GND: track 61.8 -> 121.7 mm, vias 3 -> 2
- net LED: track 0.00 -> 46.1 mm, vias 0 -> 2
- net SIDEBUTTON1: track 0.00 -> 34.4 mm
- net CAM1_EN: track 0.00 -> 29.7 mm, vias 0 -> 1
- net CAM_EN: track 28.8 -> 0.00 mm, vias 1 -> 0
- net SIDEBUTTON2: track 0.00 -> 27.1 mm, vias 0 -> 1
- net CAM2: track 23.9 -> 50.3 mm
- net SCK: track 0.00 -> 22.4 mm, vias 0 -> 1
- net ZERO_3.3V2: track 0.00 -> 19.9 mm
- net VBUS: track 19.3 -> 0.00 mm, vias 1 -> 0
- net CAM2_EN: track 0.00 -> 16.9 mm, vias 0 -> 1
- net SIDEBUTTON3: track 0.00 -> 15.7 mm
- net CAM1_OUT: track 0.00 -> 14.8 mm, vias 0 -> 1
- net ZERO_RX: track 5.72 -> 19.9 mm
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- added copper zone on layer 16, net SHIELD
Other:
- board text removed: "BAT"
- board text removed: "USB"
- board text removed: "VD1"
- board text removed: "VD2"

Commit message: controller14: production ready
Parts:
- removed D1, D3: (no value), SparkFun-LED:LED-1206
- removed U1: DS3234, SparkFun-Clocks:SO20-0.3
- R13, R3: value (none) -> 5.1k
- moved D2 41.5 mm to (25.9, 21.0)
- moved J2 41.4 mm to (19.9, 62.5)
- moved R_LED 33.4 mm to (25.7, 21.1), flipped to the bottom, turned to 180 degrees
- moved R15 10.7 mm to (10.2, 41.1), flipped to the top, turned to 90 degrees
- moved R20 8.27 mm to (7.62, 41.1), flipped to the top, turned to 90 degrees
- moved RRST 3.30 mm to (14.2, 22.4), turned to 0 degrees
- moved C5 2.54 mm to (12.3, 31.2)
- moved C4 2.34 mm to (10.0, 31.2)
- moved R1 2.09 mm to (15.7, 36.6)
- moved Q7 2.03 mm to (16.3, 32.0)
- moved Y1 1.61 mm to (11.7, 24.6)
- moved Q3 1.52 mm to (8.26, 3.94)
- moved R11 1.02 mm to (6.35, 31.4)
- moved R12 1.02 mm to (6.35, 33.8)
- moved R4 1.02 mm to (15.7, 3.56)
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Connections:
- net SHIELD renamed SHLD
- removed net BTN: U$3.12
- new net FOO9: U$3.31
- net LED: now also U$3.12; no longer U$3.31
Routing:
- net MOSI: track 7.06 -> 46.2 mm, vias 0 -> 1
- net MISO: track 12.6 -> 51.7 mm
- net RST: track 10.1 -> 46.4 mm
- net LED: track 46.1 -> 10.2 mm, vias 2 -> 1
- net SCK: track 22.4 -> 55.3 mm
- net CAM2: track 50.3 -> 36.0 mm, vias 1 -> 2
- net CAM1: track 42.6 -> 32.2 mm, vias 1 -> 2
- net N$7: track 11.9 -> 4.96 mm, vias 0 -> 1
- net N$15: track 10.8 -> 4.52 mm, vias 1 -> 0
- net VCC: track 154.2 -> 148.6 mm
- net N$19: track 9.23 -> 4.52 mm, vias 1 -> 0
- net SIDEBUTTON1: track 34.4 -> 38.2 mm
- net D+: track 5.13 -> 8.39 mm
- net ZERO_3.3V2: track 19.9 -> 17.3 mm, vias 0 -> 1
- net N$8: track 10.4 -> 13.0 mm
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Other:
- board text added: "14"
- board text removed: "+"
- board text removed: "-"
- board text removed: "12"
- board text removed: "IN"
- board text removed: "OUT"
