File: eagle/usbDirectController/usbDirectController.brd (EAGLE design)
At the start: 38.6 x 26.9 mm, 39 parts, among them IC1 MCP170312MB, J5 CORTEX_DEBUG_PTH, Q4 200mA/50V, Q8 200mA/50V, SW1 KSS221GLFS, U1 ATSAMD21G-A, U2 INA219BIDCNT, X2 ZX62D-B-5PA8, Y2 32.768kHz

Commit message: usbDirectController ready for fab
Parts:
- moved R_DLOAD 2.34 mm to (4.57, 6.86), turned to 180 degrees
- moved R2 1.85 mm to (17.0, 8.38)
- moved Q8 1.02 mm to (10.2, 6.60)
- moved R7 0.57 mm to (18.0, 7.37)
- moved C2 0.51 mm to (21.1, 9.65)
- moved R3 0.36 mm to (15.0, 7.37), turned to 0 degrees
Connections:
- net GND: now also U2.7, U2.8
- net USB_EN: now also U1.30; no longer U1.37
Routing:
- net USB_EN: track 8.73 -> 17.4 mm
- net GND: track 64.2 -> 69.9 mm, vias 8 -> 9
- net N$11: track 1.92 -> 7.05 mm
- net N$10: track 3.30 -> 6.05 mm
- net MICRO_DM: track 3.73 -> 5.21 mm
- net MICRO_VBUS: track 0.00 -> 1.30 mm, vias 0 -> 1
- net USB_5V: track 66.8 -> 66.0 mm
- net N$6: track 2.05 -> 2.66 mm
- net VCC: track 81.9 -> 82.5 mm, vias 3 -> 2
- net DM: track 25.5 -> 25.0 mm
