File: eagle/usbDirectController/usbDirectController.sch (EAGLE design)
At the start: 39 parts, among them IC1 MCP170312MB, J5 CORTEX_DEBUG_PTH, Q3 FDD4141TO252, Q4 200mA/50V, Q8 200mA/50V, SW1 KSS221GLFS, U1 ATSAMD21G-A, U2 INA219BIDCNT, X2 ZX62D-B-5PA8, Y2 32.768kHz

Commit message: usbDirectController ready for fab
Connections:
- net GND: now also U2.A0, U2.A1
- net USB_EN: now also U1.PA21(SER5:3+); no longer U1.PB22(SER5:2+)
Other:
- note removed: "voltage selection switch (USB/BATT)"
Changed lines of the file:
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@@
 <sheet>
 <plain>
-<text x="20.32" y="144.78" size="1.778" layer="91">voltage selection switch (USB/BATT)</text>
 <text x="309.88" y="233.68" size="1.778" layer="91">reverse current protection</text>
 </plain>
@@
 <instance part="J1" gate="J1" x="15.24" y="101.6" smashed="yes">
 <attribute name="VALUE" x="12.7" y="89.154" size="1.778" layer="96" font="vector" rot="MR180" align="top-left"/>
-<attribute name="NAME" x="12.7" y="112.014" size="1.778" layer="95" font="vector"/>
 </instance>
 <instance part="GND34" gate="1" x="30.48" y="78.74" smashed="yes">
@@
 </instance>
 <instance part="X2" gate="G$1" x="17.78" y="55.88" smashed="yes">
-<attribute name="NAME" x="15.24" y="67.31" size="1.778" layer="95" font="vector"/>
 <attribute name="VALUE" x="26.67" y="48.26" size="1.778" layer="96" font="vector" rot="R90"/>
 </instance>
@@
 <wire x1="53.34" y1="205.74" x2="45.72" y2="205.74" width="0.1524" layer="91"/>
 <wire x1="45.72" y1="205.74" x2="45.72" y2="203.2" width="0.1524" layer="91"/>
+<pinref part="U2" gate="G$1" pin="A0"/>
+<wire x1="53.34" y1="213.36" x2="45.72" y2="213.36" width="0.1524" layer="91"/>
+<wire x1="45.72" y1="213.36" x2="45.72" y2="210.82" width="0.1524" layer="91"/>
+<junction x="45.72" y="205.74"/>
+<pinref part="U2" gate="G$1" pin="A1"/>
+<wire x1="45.72" y1="210.82" x2="45.72" y2="205.74" width="0.1524" layer="91"/>
+<wire x1="53.34" y1="210.82" x2="45.72" y2="210.82" width="0.1524" layer="91"/>
+<junction x="45.72" y="210.82"/>
 </segment>
 <segment>
@@
 <net name="USB_EN" class="0">
 <segment>
-<pinref part="U1" gate="G$1" pin="PB22(SER5:2+)"/>
-<wire x1="330.2" y1="76.2" x2="347.98" y2="76.2" width="0.1524" layer="91"/>
-<label x="347.98" y="76.2" size="1.778" layer="95" xref="yes"/>
-</segment>
-<segment>
 <wire x1="144.78" y1="231.14" x2="144.78" y2="226.06" width="0.1524" layer="91"/>
 <pinref part="R6" gate="G$1" pin="1"/>
 <label x="144.78" y="231.14" size="1.778" layer="95" rot="R180"/>
 </segment>
-</net>
+<segment>
+<pinref part="U1" gate="G$1" pin="PA21(SER5:3+)"/>
+<wire x1="330.2" y1="106.68" x2="342.9" y2="106.68" width="0.1524" layer="91"/>
+<wire x1="342.9" y1="106.68" x2="342.9" y2="104.14" width="0.1524" layer="91"/>
+<wire x1="342.9" y1="104.14" x2="347.98" y2="104.14" width="0.1524" layer="91"/>
+<label x="347.98" y="104.14" size="1.778" layer="95" xref="yes"/>
+</segment>
+</net>

Commit message: usbDirectController2
Parts:
- C4, C5: value 22pF -> 15pF
- R3, R7: value 5.1k -> 22
- R5, RRST: value (none) -> 10k
- renumbered RRST1 to RRST
