File: eagle/usbDirectController1.5/usbDirectController1.5.sch (EAGLE design)
At the start: 39 parts, among them IC1 MCP170312MB, J5 CORTEX_DEBUG_PTH, Q3 FDD4141TO252, Q4 200mA/50V, Q8 200mA/50V, SW1 KSS221GLFS, U1 ATSAMD21G-A, U2 INA219BIDCNT, X2 ZX62D-B-5PA8, Y2 32.768kHz

Commit message: usbDirectController sent to fab
Parts:
- removed C9: 100uF, SparkFun-Capacitors:100UF-POLAR-25V-20%(ELEC)
- removed J3: (no value), SparkFun-Connectors:CONN_04
- removed Q3: FDD4141TO252, transistor-fet:FDD4141TO252
- removed Q4: 200mA/50V, SparkFun-DiscreteSemi:MOSFET-NCHANNELBSS138
- removed R1: ?, SparkFun-Passives:RESISTOR2010
- removed R3, R7: 22, SparkFun-Passives:RESISTOR0805-RES
- removed R4: 10k, SparkFun-Resistors:RESISTOR0805-RES
- removed R6: 1k, SparkFun-Resistors:RESISTOR0805-RES
- removed RPU1, RPU2: 10k, SparkFun-Passives:RESISTOR0805-RES
- removed U2: INA219BIDCNT, microbuilder:INA219
- added AP2553: MCP4725, SparkFun-IC-Conversion:MCP4725SOT-23
- added C10: 10uF, SparkFun-Capacitors:1.0UF-0805-25V-10%
- added C11: 0.1uF, SparkFun-Capacitors:1.0UF-0805-25V-10%
- added C12: 1.0uF, SparkFun-Capacitors:1.0UF-1206-50V-10%
- added C13: 120uF, SparkFun-Capacitors:1.0UF-1206-50V-10%
- added MCP9808: V_REG_MIC5216, SparkFun-IC-Power:V_REG_MIC5216
- added R_I2C_1, R_I2C_2, R_MOSFET_USB2, R_MOSFET_USB3, R_MOSFET_USB4: 10k, SparkFun-Passives:RESISTOR0805-RES
- added R_MOSFET_USB1: ? (1%), SparkFun-Passives:RESISTOR0805-RES
- C1: value 1.0uF -> 0.1uF
- C8: device SparkFun-Capacitors:1.0UF-0805-25V-10% -> SparkFun-Capacitors:1.0UF-1206-50V-10%
Connections:
- removed net MOSFET_OUT: Q3.D, R1.1, U2.VIN-
- removed net N$6: R3.2, X2G$1.2
- removed net N$9: R7.2, X2G$1.3
- removed net OUT_5V: C9.+, R1.2, U2.VIN+, USB_1.VBUS
- removed net USB_EN: R6.1, U1.PA21(SER5:3+)
- new net N$5: AP2553.SDA, R_MOSFET_USB2.1, R_MOSFET_USB4.1
- new net USB1_EN: AP2553.VDD, R_MOSFET_USB3.2, U1.PA21(SER5:3+)
- new net USB1_OUT: AP2553.AO, C12.2, C13.2, USB_1.VBUS
- new net USB2_EN: U1.PA19(SER1:3+)
- new net USB_FAULT: R_MOSFET_USB4.2, U1.PB23(SER5:3+)
- net DM: no longer J3.2
- net DP: no longer J3.3
- net GND: now also AP2553.VSS, C1.2, C10.2, C11.2, C12.1, C13.1, MCP9808.FLAG, MCP9808.GND@5, MCP9808.GND@6, MCP9808.GND@7, R_MOSFET_USB1.1, R_MOSFET_USB2.2, R_MOSFET_USB3.1; no longer C1.1, C9.-, J3.1, Q4.S, U2.A0, U2.A1, U2.GND
- net MICRO_DM: now also X2G$1.2; no longer R3.1
- net MICRO_DP: now also X2G$1.3; no longer R7.1
- net N$2: now also MCP9808.VOUT; no longer Q4.G, R6.2
- net N$3: now also AP2553.SCL, R_MOSFET_USB1.2; no longer Q3.G, Q4.D, R4.2
- net SCL: now also MCP9808.VIN, R_I2C_1.2; no longer RPU1.1, U2.SCL
- net SDA: now also MCP9808.EN, R_I2C_2.1; no longer RPU2.2, U2.SDA
- net USB_5V: now also AP2553.VOUT, C10.1, C11.1; no longer J3.4, Q3.S, R4.1
- net VCC: now also C1.1, MCP9808.GND@8, R_I2C_1.1, R_I2C_2.2; no longer C1.2, RPU1.2, RPU2.1, U2.VCC
Other:
- note added: "AP2553"
- moved on the sheet: C1, C8
