File: eagle/usbDirectController1.6/usbDirectController1.6.brd (EAGLE design)
At the start: 30 x 65 mm, 53 parts, among them IC1 MCP170312MB, IC3 FE1.1S, Q2 200mA/50V, Q4 200mA/50V, Q6 200mA/50V, Q8 200mA/50V, U1 ATSAMD21G-A, X2 ZX62D-B-5PA8, Y2 32.768

Commit message: minor changes in schematics
Parts:
- removed C9: 100uF, SparkFun-Capacitors:PANASONIC_D
- removed H1, H2, H3, H4: MOUNT-HOLE2.8, holes:2,8
- removed IC3: FE1.1S, FE1.1S:SOP64P600X175-28N
- removed J2: (no value), SparkFun-Connectors:1X04
- removed J6, J7, J8: (no value), SparkFun-Connectors:1X01_POGOPIN_HOLE_0.58_DIA
- removed Q1, Q3, Q5, Q7: (no value), transistor-fet:TO252
- removed Q2, Q4, Q6: 200mA/50V, SparkFun-DiscreteSemi:SOT23-3
- removed R10, R12, R6, R8: 1k, SparkFun-Resistors:1206
- removed R11, R4, R7, R9: 10k, SparkFun-Resistors:1206
- removed REXT: 2.7k, SparkFun-Passives:1206
- removed RRST1: (no value), SparkFun-Passives:1206
- removed S1: TAC_SWITCHSMD, SparkFun-Retired:TACTILE-PTH
- removed U$4: NANOFIT2, volzolib:NANOFIT2
- removed USB_2, USB_3: USB_A_SMT_FEMALE, SparkFun-Connectors:USB-A-S-SILK-FEMALE
- removed Y1: (no value), SparkFun-FreqCtrl:CRYSTAL-SMD-5X3
- added AP2553: MCP4725, SparkFun-IC-Conversion:SOT23-6
- added C10: 10uF, SparkFun-Capacitors:0805
- added C11: 0.1uF, SparkFun-Capacitors:0805
- added C12: 1.0uF, SparkFun-Capacitors:1206
- added C13: 120uF, SparkFun-Capacitors:1206
- added H5, H8: MOUNT-HOLE2.8, holes:2,8
- added MCP9808: V_REG_MIC5216, SparkFun-IC-Power:MSOP8
- added R2: 1k, SparkFun-Resistors:0805
- added RRST, R_I2C_1, R_I2C_2, R_MOSFET_USB2, R_MOSFET_USB3, R_MOSFET_USB4: 10k, SparkFun-Passives:0805
- added R_DLOAD: 1k, SparkFun-Resistors:1206
- added R_MOSFET_USB1: ? (1%), SparkFun-Passives:0805
- added SW1: KSS221GLFS, adafruit:BTN_CK_KSS
- C1, C2, C3, C6: value 100uF -> 0.1uF; device SparkFun-Capacitors:PANASONIC_D -> SparkFun-Capacitors:0805
- C4, C5: value 22pF -> 15pF; device SparkFun-Passives:1206 -> SparkFun-Passives:0805
- C7: device SparkFun-Capacitors:1206 -> SparkFun-Capacitors:0805
- J5: value (none) -> CORTEX_DEBUG_PTH; device SparkFun-Connectors:1X01_POGOPIN_HOLE_0.58_DIA -> SparkFun-Connectors:2X5-PTH-1.27MM
- R5: value (none) -> 10k; device SparkFun-Passives:1206 -> SparkFun-Passives:0805
- R_LED: device SparkFun-Resistors:1206 -> SparkFun-Resistors:0805
- Y2: value 32.768 -> 32.768kHz; device SparkFun-FreqCtrl:CRYSTAL-SMD-5X3 -> samd21-temp:CRYSTAL-SMD-3.2X1.5MM
- moved Q8 103.7 mm to (2.54, 3.56), flipped to the bottom, turned to 270 degrees
- moved X2 50.3 mm to (14.2, 0.00), turned to 90 degrees
- moved D2 47.1 mm to (3.17, 4.06), turned to 270 degrees
- moved C6 44.6 mm to (23.6, 17.3), flipped to the bottom, turned to 90 degrees
- moved C7 41.8 mm to (6.10, 20.3), turned to 180 degrees
- moved R5 40.4 mm to (40.6, 5.59), turned to 270 degrees
- moved C4 38.9 mm to (20.6, 21.0), flipped to the top, turned to 180 degrees
- moved IC1 37.8 mm to (6.10, 23.9), turned to 180 degrees
- moved USB_1 35.6 mm to (27.9, 13.7)
- moved C8 34.7 mm to (6.10, 22.9), flipped to the top
- moved U1 33.7 mm to (15.7, 13.7), turned to 270 degrees
- moved C5 33.2 mm to (21.3, 25.3), flipped to the top, turned to 180 degrees
- moved J5 26.7 mm to (18.3, 32.0), turned to 180 degrees
- moved R_LED 17.1 mm to (7.62, 2.29), turned to 270 degrees
- moved C3 14.6 mm to (16.8, 21.1), turned to 180 degrees
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Connections:
- removed net BATT_VCC: U$4.P$2
- removed net CONV_5V: IC3.20
- removed net HUB1: C9.+, USB_1.VBUS
- removed net HUB2: C1.+, USB_2.VBUS
- removed net HUB3: C2.+, USB_3.VBUS
- removed net HUB_1: Q3.3
- removed net HUB_1_EN: R6.1
- removed net HUB_2: Q1.3
- removed net HUB_2_EN: R10.1
- removed net HUB_3: Q5.3
- removed net HUB_3_EN: R8.1
- removed net HUB_ZERO: C6.+, Q7.3
- removed net HUB_ZERO_EN: R12.1
- removed net MICRO_ID: X2.4
- removed net N$12: Q5.1, Q6.3, R7.2
- removed net N$13: Q6.1, R8.2
- removed net N$15: Q7.1, Q8.3, R11.2
- removed net N$19: Q8.1, R12.2
- removed net N$21: RRST1.1, U1.40
- removed net N$23: IC3.3, Y2.1
- removed net N$24: IC3.2, Y2.3
- removed net N$31: IC3.14, REXT.2
- removed net N$6: Q2.1, R10.2
- removed net UC_DM: IC3.10, U1.33
- removed net UC_DP: IC3.11, U1.34
- removed net USB_1_DM: IC3.8, USB_1.D-
- removed net USB_1_DP: IC3.9, USB_1.D+
- removed net USB_2_DM: IC3.6, USB_2.D-
- removed net USB_2_DP: IC3.7, USB_2.D+
- removed net USB_3_DM: IC3.4, USB_3.D-
- removed net USB_3_DP: IC3.5, USB_3.D+
- removed net VCC_5V: C7.1, IC1.2@1, Q1.2, Q3.2, Q5.2, Q7.2, R11.1, R4.1, R7.1, R9.1
- removed net ZERO_DM: IC3.15, J1.A7, J1.B7, J8.1
- removed net ZERO_DP: IC3.16, J1.A6, J1.B6, J7.1
- new net DM: J1.A7, J1.B7, USB_1.D-
- new net DP: J1.A6, J1.B6, USB_1.D+
- new net DUMMY_LOAD: R2.1, U1.27
- new net N$10: Q8.1, R2.2
- new net N$11: Q8.3, R_DLOAD.1
- new net N$5: AP2553.4, R_MOSFET_USB2.1, R_MOSFET_USB4.1
- new net RESET: J5.10, RRST.1, U1.40
- new net SCL: MCP9808.2, R_I2C_1.2, U1.32
- new net SDA: MCP9808.1, R_I2C_2.1, U1.31
- new net USB1_EN: AP2553.3, R_MOSFET_USB3.2, U1.30
- new net USB1_OUT: AP2553.6, C12.2, C13.2, USB_1.VBUS
- new net USB2_EN: U1.28
- new net USB_FAULT: R_MOSFET_USB4.2, U1.38
- net BTN: now also SW1.P$2, U1.25; no longer S1.4
- net GND: now also AP2553.2, C1.2, C10.2, C11.2, C12.1, C13.1, C2.1, C3.1, C6.2, J5.3, J5.5, MCP9808.4, MCP9808.5, MCP9808.6, MCP9808.7, R_MOSFET_USB1.1, R_MOSFET_USB2.2, R_MOSFET_USB3.1, SW1.P$1, U1.5; no longer C1.-, C2.-, C3.-, C6.-, C9.-, IC3.1, J2.1, Q2.2, Q4.2, Q6.2, REXT.1, S1.2, U$4.P$1, USB_2.GND, USB_3.GND
- net LED: now also U1.26
- net MICRO_DM: now also U1.33
- net MICRO_DP: now also U1.34
- net N$1: now also C6.1, U1.43; no longer Q1.1, Q2.3, R9.2
- net N$2: now also MCP9808.3; no longer Q4.1, R6.2
- net N$3: now also AP2553.5, R_MOSFET_USB1.2; no longer Q3.1, Q4.3, R4.2
- net N$32: now also Y2.P$1; no longer Y1.1
- net N$8: now also Y2.P$2; no longer Y1.3
- net SWDCLK: now also J5.4; no longer J2.2
- net SWDIO: now also J5.2; no longer J2.3
- net USB_5V: now also AP2553.1, C10.1, C11.1, C7.1, IC1.2@1, R_DLOAD.2; no longer C3.+
- net VCC: now also C1.1, C2.2, C3.2, J5.1, MCP9808.8, RRST.2, R_I2C_1.1, R_I2C_2.2; no longer J2.4, RRST1.2, U1.43
Routing:
- net DP: track 0.00 -> 25.7 mm
- net DM: track 0.00 -> 16.8 mm
- net GND: track 9.75 -> 0.00 mm, vias 18 -> 0
- net USB_3_DM: track 8.65 -> 0.00 mm
- net USB_5V: track 7.76 -> 0.00 mm
- net USB_3_DP: track 7.44 -> 0.00 mm
- net CC1: track 7.24 -> 0.00 mm, vias 1 -> 0
- net CC2: track 7.02 -> 0.00 mm, vias 1 -> 0
- net MICRO_DM: track 0.00 -> 6.23 mm, vias 0 -> 1
- net MICRO_DP: track 0.00 -> 5.16 mm, vias 0 -> 1
- added copper zone on layer 16, net SHLD
- added copper zone on layer 16, net USB1_OUT
- removed copper zone on layer 1, net GND
- removed copper zone on layer 1, net HUB2
- removed copper zone on layer 1, net HUB3
- removed copper zone on layer 16, net HUB3
- removed copper zone on layer 1, net USB_5V
Other:
- board size 30 x 65 mm -> 5.6 x 9.2 mm
- board text added: "UDC 1.5"
- board text removed: "+"
- board text removed: "-"
- board text removed: "12"
- board text removed: "BOX"
- board text removed: "TIME"
