File: eagle/usbDirectController1.6/usbDirectController1.6.sch (EAGLE design)
At the start: 39 parts, among them IC1 MCP170312MB, J5 CORTEX_DEBUG_PTH, Q8 200mA/50V, SW1 KSS221GLFS, U1 ATSAMD21G-A, X2 ZX62D-B-5PA8, Y2 32.768kHz

Commit message: minor changes in schematics
Other:
- moved on the sheet: MCP9808, Q8, R13, R14, R2, R_DLOAD
