File: eagle/controller11_2/controller11_2.sch (EAGLE design)
At the start: 62 parts, among them IC1 ILD213T, IC2 MCP170312MB, J3 CONN_20X2, J5 CORTEX_DEBUG_PTH, Q1 FDD4141TO252, Q2 200mA/50V, SW1 KSS221GLFS, U2 ATSAMD21G-A, U3 MP2307, X1 1501_04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

Commit message: progress controller11_2
Parts:
- removed J3: CONN_20X2, SparkFun-Connectors:CONN_20X2
- removed U$4, U$5: NANOFIT2, volzolib:NANOFIT2
- added J1, J2: POWER_JACKPTH_BREAD, SparkFun-Connectors:POWER_JACKPTH_BREAD
- added JP2: (no value), adafruit:PINHD-2X20
- added RBTN1: 10k, SparkFun-Passives:RESISTOR0805-RES
- added SW2: KSS221GLFS, adafruit:SWITCH_PUSHBUTTONC&K_KSS
- R_LED: device SparkFun-Resistors:RESISTOR1206 -> SparkFun-Resistors:RESISTOR0805-RES
Connections:
- net USB1_EN renamed ZERO_EN
- removed net BTN: RBTN.2, SW1.P$2, U2.PA16(I2C/SER1:0+)
- removed net USB1_OUT: AP2553.AO, C3.2, C4.2
- removed net USB2_EN: U2.PA19(SER1:3+)
- removed net USB_5V: AP2553.VOUT, C1.1, C2.1, C7.1, IC2.VI1
- new net BTN1: RBTN.2, SW1.P$2, U2.PA15(XOUT/SER2:3+)
- new net BTN2: RBTN1.2, SW2.P$2, U2.PA16(I2C/SER1:0+)
- net BATT_VCC: now also J1.PWR; no longer U$4.LEFT
- net CAM1: now also U2.PA05(AIN5/SER0:1/TC0:1)
- net CAM2: now also U2.PA06(AIN6/SER0:2/TC1:0)
- net CAM_EN: now also U2.PB02(AIN10/SER5:0)
- net CAM_OUT: now also J2.PWR; no longer U$5.LEFT
- net CONV_5V: now also AP2553.VOUT, C1.1, C2.1, C7.1, IC2.VI1
- net GND: now also J1.GND, J2.GND, JP2.6, SW2.P$1; no longer J3.6, U$4.RIGHT, U$5.RIGHT
- net VCC: now also RBTN1.1
- net VD_DIRECT: now also U2.PB08(AIN2/SER4:0/TC4:0)
- net ZERO_5V: now also AP2553.AO, C3.2, C4.2, JP2.2; no longer J3.2
- net ZERO_RX: now also JP2.10, U2.PA10(AIN18/SER0:2+); no longer J3.10
- net ZERO_TX: now also JP2.8, U2.PA11(AIN19/SER0:3+); no longer J3.8

Commit message: additional eagle boards
Parts:
- removed C1: 10uF, SparkFun-Capacitors:1.0UF-0805-25V-10%
- added C22: 120uF, SparkFun-Capacitors:1.0UF-1206-50V-10%
Connections:
- net CONV_5V: now also C22.1; no longer C1.1
- net GND: now also C22.2; no longer C1.2
- net VD_DIRECT: now also U2.PA07(AIN7/SER0:3/TC1:1); no longer U2.PB08(AIN2/SER4:0/TC4:0)
