File: eagle/usbDirectController3/usbDirectController3.brd (EAGLE design)
At the start: 37.6 x 22.4 mm, 37 parts, among them IC1 MCP170312MB, J1 USB_A_SMT_MALE, J5 CORTEX_DEBUG_PTH, Q4 200mA/50V, U1 ATSAMD21G-A, Y2 32.768kHz

Commit message: UDC3 bugfixes
Parts:
- C4, C5: value 15pF -> 22pF
- C6: value 0.1uF -> 1.0uF
- R_LED: value 4.7k -> 470
Changed lines of the file:
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@@
 </autorouter>
 <elements>
-<element name="C4" library="SparkFun-Passives" package="0805" value="15pF" x="21.082" y="15.367" smashed="yes" rot="MR180"/>
-<element name="C5" library="SparkFun-Passives" package="0805" value="15pF" x="21.971" y="12.7" smashed="yes" rot="MR90"/>
+<element name="C4" library="SparkFun-Passives" package="0805" value="22pF" x="21.082" y="15.367" smashed="yes" rot="MR180"/>
+<element name="C5" library="SparkFun-Passives" package="0805" value="22pF" x="21.971" y="12.7" smashed="yes" rot="MR90"/>
 <element name="D2" library="SparkFun-LED" package="WS2812B" value="" x="14.986" y="11.303" smashed="yes" rot="R180">
 <attribute name="PROD_ID" value="DIO-12503" x="14.986" y="11.303" size="1.778" layer="27" rot="R180" display="off"/>
 <attribute name="VALUE" x="10.732" y="12.903" size="0.6096" layer="27" rot="R180"/>
 </element>
-<element name="R_LED" library="SparkFun-Resistors" package="0805" value="4.7k" x="9.144" y="7.874" smashed="yes" rot="R180"/>
+<element name="R_LED" library="SparkFun-Resistors" package="0805" value="470" x="9.144" y="7.874" smashed="yes" rot="R180"/>
 <element name="R5" library="SparkFun-Passives" package="0805" value="10k" x="10.668" y="1.524" smashed="yes">
 <attribute name="VALUE" x="9.271" y="0" size="0.4064" layer="27"/>
@@
 <attribute name="VALUE" x="8.382" y="15.621" size="0.6096" layer="28" font="vector" ratio="20" rot="MR180" align="top-center"/>
 </element>
-<element name="C6" library="SparkFun-Capacitors" library_urn="urn:adsk.eagle:library:510" package="0805" package3d_urn="urn:adsk.eagle:package:37429/1" value="0.1uF" x="15.748" y="18.034" smashed="yes" rot="MR90">
+<element name="C6" library="SparkFun-Capacitors" library_urn="urn:adsk.eagle:library:510" package="0805" package3d_urn="urn:adsk.eagle:package:37429/1" value="1.0uF" x="15.748" y="18.034" smashed="yes" rot="MR90">
 <attribute name="PROD_ID" value="CAP-08064" x="15.748" y="18.034" size="1.778" layer="28" rot="MR90" display="off"/>
 <attribute name="VALUE" x="14.859" y="18.034" size="0.6096" layer="28" font="vector" ratio="20" rot="MR90" align="top-center"/>
