File: eagle/controller15/controller15.sch (EAGLE design)
At the start: 77 parts, among them IC1 MCP170312MB, IC3 FE1.1S, J2 CORTEX_DEBUG_PTH, J3 POWER_JACKPTH_BREAD, J4 POWER_JACKPTH_BREAD, Q3 FDD4141TO252, Q4 200mA/50V, U1 ATSAMD21G-A, U3 MP2307, X2 ZX62D-B-5PA8, Y1 32.768kHz, Y2 32.768kHz

Commit message: controller15 sent to fab
Parts:
- removed C26: 4.7uF, SparkFun-Capacitors:1.0UF-1206-50V-10%
- removed C27: 10uF, SparkFun-Capacitors:1.0UF-1206-50V-10%
- removed L1: 2.2µH/±20%/1.5A, SparkFun-Coils:INDUCTOR-VLF4012AT-2.2UH
- removed LM3671: MCP73811/2, adafruit:MCP73811/2
- removed R21: (no value), SparkFun-Passives:RESISTOR0805-RES
- added C28, C29: 10uF, SparkFun-Capacitors:1.0UF-0805-25V-10%
- added R7: 10k, SparkFun-Passives:RESISTOR0805-RES
- REXT: value 2.7k -> 2.7k / 1%
- Y2: value 32.768kHz -> 12MHz
Connections:
- removed net EN: LM3671.VBAT, R21.1
- removed net N$1: L1.1, LM3671.PROG
- new net N$15: IC3.XRSTJ, R7.1
- new net VD_18: C28.1, IC3.VD18, IC3.VD18_O
- new net VD_33: C29.2, IC3.BUSJ, IC3.OVCJ, IC3.VD33, IC3.VD33_O, R7.2
- net CAM_EN: now also U1.PA05(AIN5/SER0:1/TC0:1); no longer U1.PB03(AIN11/SER5:1)
- net CONV_5V: no longer C26.2, LM3671.CE, R21.2
- net GND: now also C28.2, C29.1, IC3.TESTJ; no longer C26.1, C27.2, LM3671.VSS
- net LED: now also U1.PA18(SER1:2+); no longer U1.PA10(AIN18/SER0:2+)
- net USB1_EN: now also U1.PA21(SER5:3+); no longer U1.PB23(SER5:3+)
- net VCC: no longer C27.1, L1.2, LM3671.VDD
Other:
- note removed: "(ADC for external battery)"
- note removed: "RTC"
- note removed: "Reverse Current Protection"
- note removed: "connect vd33_O and vd33??"
- note removed: "correct crystal??"
- note removed: "is it really clever to use the enable pin to disable battery input?"
- note removed: "reverse current protection"
- note removed: "temperature sensor"
- moved on the sheet: REXT

Commit message: new PCB files (batteryholder, templog2, ...)
Connections:
- net GND: no longer IC3.TESTJ
Changed lines of the file:
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@@
 <part name="GND40" library="SparkFun-Aesthetics" deviceset="GND" device=""/>
 <part name="R7" library="SparkFun-Passives" deviceset="RESISTOR" device="0805-RES" value="10k"/>
-<part name="GND42" library="SparkFun-Aesthetics" deviceset="GND" device=""/>
 </parts>
 <sheets>
@@
 <attribute name="NAME" x="171.2214" y="80.01" size="1.778" layer="95" rot="R90"/>
 <attribute name="VALUE" x="176.022" y="80.01" size="1.778" layer="96" rot="R90"/>
-</instance>
-<instance part="GND42" gate="1" x="152.4" y="111.76" smashed="yes" rot="R180">
-<attribute name="VALUE" x="154.94" y="114.3" size="1.778" layer="96" rot="R180"/>
 </instance>
 </instances>
@@
 <wire x1="167.64" y1="99.06" x2="167.64" y2="101.6" width="0.1524" layer="91"/>
 </segment>
-<segment>
-<pinref part="IC3" gate="G$1" pin="TESTJ"/>
-<wire x1="124.46" y1="104.14" x2="152.4" y2="104.14" width="0.1524" layer="91"/>
-<wire x1="152.4" y1="104.14" x2="152.4" y2="109.22" width="0.1524" layer="91"/>
-<pinref part="GND42" gate="1" pin="GND"/>
-</segment>
 </net>
