File: eagle/zerocam2S/zerocam2S.brd (EAGLE design)
At the start: 30.7 x 65 mm, 48 parts, among them IC1 MCP170312MB, J5 CORTEX_DEBUG_PTH, U1 ATSAMD21G-A, U3 MP2307, X2 ZX62D-B-5PA8, Y2 32.768kHz

Commit message: new PCB files (batteryholder, templog2, ...)
Parts:
- moved J1 0.51 mm to (14.7, 3.68)
- moved X2 0.13 mm to (30.6, 53.3)
Routing:
- net GNDA: track 27.7 -> 31.8 mm
- net BATT_VCC: track 35.5 -> 34.9 mm
Other:
- board text added: "+"
- board text added: "-"
- board text added: "ver. 1"
- board text added: "zerocam2S1P"
