File: eagle/batteryholder286P_vertical/batteryholder2S6P_vertical.brd (EAGLE design)
At the start: 84.5 x 34.5 mm, 1 part

Commit message: batteryholder boards minor changes
Changed lines of the file:
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@@
 <?xml version="1.0" encoding="utf-8"?>
 <!DOCTYPE eagle SYSTEM "eagle.dtd">
-<eagle version="9.5.0">
+<eagle version="9.5.1">
 <drawing>
 <settings>
@@
 <text x="18.5" y="19.5" size="1.778" layer="22" rot="MR0" align="center">2</text>
 <text x="2" y="22" size="1" layer="21" align="top-left">2S4P</text>
-<text x="1.9" y="19" size="1" layer="21" align="top-left">vertical</text>
-<text x="1.9" y="20.5" size="1" layer="21" align="top-left">rev. A</text>
+<text x="1.9" y="20.5" size="1" layer="21" align="top-left">vertical</text>
+<text x="1.9" y="19" size="1" layer="21" align="top-left">rev. A</text>
 <circle x="80.5" y="9" radius="2" width="0.1524" layer="21"/>
 <circle x="4" y="25.5" radius="2" width="0.1524" layer="21"/>
