File: eagle/batteryholder286P_vertical_2/batteryholder2S6P_vertical_2.brd (EAGLE design)
At the start: 84.5 x 34.5 mm, 2 parts, among them J2 5.5x2.1mm Barrel

Commit message: batteryholder boards minor changes
Parts:
- added J3: (no value), SparkFun-Connectors:SCREWTERMINAL-5MM-3
- moved J2 1.00 mm to (3.50, 14.5)
Connections:
- new net N$3: J1.1, J3.2
- net B+: now also J3.3
- net B-: now also J3.1
Routing:
- net B-: track 0.00 -> 35.6 mm, vias 0 -> 46
- net N$3: track 0.00 -> 21.8 mm
- added copper zone on layer 1, net B+
- added copper zone on layer 16, net B+
- added copper zone on layer 1, net B-
- added copper zone on layer 16, net B-
- removed copper zone on layer 16, net N$1
- removed copper zone on layer 16, net N$2
Other:
- board text removed: "BOTTOM"
- board text removed: "TOP"
- board text removed: "all connected"
- board text removed: "pairs connected"
