File: eagle/batteryholder2S3P/batteryholder2S3P.sch (EAGLE design)
At the start: 3 parts, among them J2 5.5x2.1mm Barrel

Commit message: batteryholder boards minor changes
Parts:
- removed J2: 5.5x2.1mm Barrel, SparkFun-Connectors:POWER_JACKSMD
- added BT1, BT2, BT3: KEYSTONE_1048KEYSTONE_1048_0_0, Keystone - 1048:KEYSTONE_1048KEYSTONE_1048_0_0
- added H1, H2, H3, H4: MOUNT-HOLE3.2, holes:MOUNT-HOLE3.2
- J1: device SparkFun-Connectors:CONN_01PTH_2MM -> SparkFun-Connectors:CONN_03-SCREW-5MM
- J3: value (none) -> 5.5x2.1mm Barrel; device SparkFun-Connectors:CONN_03-SCREW-5MM -> SparkFun-Connectors:POWER_JACKSMD
Connections:
- removed net B+: J2.PWR, J3.3
- removed net B-: J2.GND, J2.GNDBREAK, J3.1
- removed net N$3: J1.1, J3.2
- new net BOTTOM_MINUS: BT1A.1_CATHODE, BT1B.2_ANODE, BT2A.1_CATHODE, J1.1, J3.GND
- new net TOP_MINUS: BT1A.1_ANODE, BT1B.2_CATHODE, BT2A.1_ANODE, BT2B.2_CATHODE, BT3A.1_ANODE, BT3B.2_CATHODE, J1.2
- new net TOP_PLUS: BT2B.2_ANODE, BT3A.1_CATHODE, BT3B.2_ANODE, J1.3, J3.PWR
