File: eagle/controller15_2/controller15_2.brd (EAGLE design)
At the start: 30 x 65 mm, 64 parts, among them IC1 ILD213T, IC2 MCP170312MB, J1 POWER_JACKPTH_BREAD, J2 POWER_JACKPTH_BREAD, J5 CORTEX_DEBUG_PTH, Q2 200mA/50V, SW1 KSS221GLFS, SW2 KSS221GLFS, U2 ATSAMD21G-A, U3 MP2307, X1 1501_04, X2 ZX62D-B-5PA8, Y2 32.768kHz

Commit message: additional eagle boards
Parts:
- removed IC2: MCP170312MB, linear:SOT89
- removed J1: POWER_JACKPTH_BREAD, SparkFun-Connectors:POWER_JACK_PTH_BREAD
- removed J5: CORTEX_DEBUG_PTH, SparkFun-Connectors:2X5-PTH-1.27MM
- removed JP1: (no value), SparkFun-Passives:PAD-JUMPER-2-NO_YES_SILK
- removed JP2: (no value), adafruit:2X20
- removed Q1: (no value), transistor-fet:TO252
- removed Q2: 200mA/50V, SparkFun-DiscreteSemi:SOT23-3
- removed R10: 1k, SparkFun-Resistors:0805
- removed R15, R20: (no value), SparkFun-Passives:0805
- removed R9: 10k, SparkFun-Resistors:0805
- removed RBTN, RBTN1: 10k, SparkFun-Passives:0805
- removed SW1, SW2: KSS221GLFS, adafruit:BTN_CK_KSS
- removed U2: ATSAMD21G-A, SparkFun-IC-Microcontroller:TQFP-48
- removed X1: 1501_04, con-lumberg:1501_05
- added AP1, AP2: MCP4725, SparkFun-IC-Conversion:SOT23-6
- added C1: 0.1uF, SparkFun-Capacitors:0805
- added C23: 1.0uF, SparkFun-Capacitors:1206
- added C24: 120uF, SparkFun-Capacitors:1206
- added C25: 1.0uF, SparkFun-Capacitors:0805
- added C28, C29: 10uF, SparkFun-Capacitors:0805
- added D1: 3A/40V/500mV, SparkFun-DiscreteSemi:SMA-DIODE
- added IC3: FE1.1S, FE1.1S:SOP64P600X175-28N
- added J3, J4: POWER_JACKPTH_BREAD, SparkFun-Connectors:POWER_JACK_PTH_BREAD
- added Q3: (no value), transistor-fet:TO252
- added Q4: 200mA/50V, SparkFun-DiscreteSemi:SOT23-3
- added R4: 10k, SparkFun-Resistors:0805
- added R5: (no value), SparkFun-Passives:0805
- added R6: 1k, SparkFun-Resistors:0805
- added R7, R_MOSFET_USB4, R_MOSFET_USB6: 10k, SparkFun-Passives:0805
- added REXT: 2.7k / 1%, SparkFun-Passives:0805
- added R_MOSFET_USB2, R_MOSFET_USB5: ? (1%), SparkFun-Passives:0805
- added S1: TAC_SWITCHSMD, SparkFun-Retired:TACTILE-SWITCH-SMD
- added U1: ATSAMD21G-A, SparkFun-IC-Microcontroller:TQFP-48
- added USB_1, USB_2: USB_A_SMT_FEMALE, SparkFun-Connectors:USB-A-S-SILK-FEMALE
- added Y1: 32.768kHz, SparkFun-FreqCtrl:CRYSTAL-SMD-3.2X1.5MM
- C10: value 15pF -> 10uF; device SparkFun-Passives:0805 -> SparkFun-Capacitors:1206
- C11: value 15pF -> 0.1uF; device SparkFun-Passives:0805 -> SparkFun-Capacitors:0805
- C12: value 0.1uF -> 1.0uF; device SparkFun-Capacitors:0805 -> SparkFun-Capacitors:1206
- C13: device SparkFun-Capacitors:1206 -> SparkFun-Capacitors:0805
- C17: value 22uF / 6.3V -> 0.1uF; device SparkFun-Capacitors:1210 -> SparkFun-Capacitors:0805
- C18: value 10uF / 25V -> 1.0uF; device SparkFun-Capacitors:1210 -> SparkFun-Capacitors:1206
- C2, C20: value 0.1uF -> 120uF; device SparkFun-Capacitors:0805 -> SparkFun-Capacitors:1206
- C21: value 0.1uF -> 10uF; device SparkFun-Capacitors:0805 -> SparkFun-Capacitors:1206
- C22: value 120uF -> 0.1uF; device SparkFun-Capacitors:1206 -> SparkFun-Capacitors:0805
- C3: value 1.0uF -> 10uF; device SparkFun-Capacitors:0805 -> SparkFun-Capacitors:1206
- C4: value 120uF -> 22pF; device SparkFun-Capacitors:1206 -> SparkFun-Passives:0805
- C5: value 100uF -> 22pF; device SparkFun-Capacitors:PANASONIC_D -> SparkFun-Passives:0805
- C7: device SparkFun-Capacitors:0805 -> SparkFun-Capacitors:1206
- IC1: value ILD213T -> MCP170312MB; device SparkFun-DiscreteSemi:SO08 -> linear:SOT89
- J2: value POWER_JACKPTH_BREAD -> CORTEX_DEBUG_PTH; device SparkFun-Connectors:POWER_JACK_PTH_BREAD -> SparkFun-Connectors:2X5-PTH-1.27MM
- RRST1: value 10k -> (none)
- R_LED: value 4.7k -> 470
- Y2: value 32.768kHz -> 12MHz; device samd21-temp:CRYSTAL-SMD-3.2X1.5MM -> SparkFun-FreqCtrl:CRYSTAL-SMD-5X3
- moved C3 55.9 mm to (9.65, 59.7), flipped to the top, turned to 180 degrees
- moved C20 54.4 mm to (19.8, 61.5)
- moved R2 53.2 mm to (8.51, 3.68), flipped to the top, turned to 270 degrees
- moved R24 52.6 mm to (17.5, 2.29), flipped to the top, turned to 180 degrees
- moved C15 49.6 mm to (18.5, 4.83), turned to 180 degrees
- moved R1 46.5 mm to (12.4, 2.29), flipped to the top, turned to 180 degrees
- moved U3 46.3 mm to (14.7, 10.2)
- moved C13 45.8 mm to (17.3, 15.9), turned to 90 degrees
- moved C22 45.2 mm to (7.11, 57.4), flipped to the top
- moved C14 43.9 mm to (12.4, 4.83), flipped to the top, turned to 0 degrees
- moved C16 43.6 mm to (4.83, 12.1), turned to 180 degrees
- moved C19 43.1 mm to (14.0, 15.7)
- moved X2 41.5 mm to (0.00, 41.4), turned to 0 degrees
- moved Y2 40.9 mm to (13.7, 56.6), flipped to the bottom, turned to 0 degrees
- moved C21 36.5 mm to (10.2, 55.9), turned to 270 degrees
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Connections:
- removed net BTN1: RBTN.2, SW1.P$2, U2.24
- removed net BTN2: RBTN1.2, SW2.P$2, U2.25
- removed net CAM1: R20.1, U2.10
- removed net CAM2: R15.1, U2.11
- removed net N$1: Q1.1, Q2.3, R9.2
- removed net N$12: IC1.6, X1.2
- removed net N$13: IC1.8, X1.3
- removed net N$19: IC1.1, R20.2
- removed net N$34: IC1.5, IC1.7, JP1.2, X1.1
- removed net N$6: Q2.1, R10.2
- removed net USB_FAULT: U2.38
- removed net VD_DIRECT: C6.1, U2.12, VD1.1, VD2.2
- removed net ZERO_5V: AP2553.6, C3.2, C4.2, JP2.2
- removed net ZERO_EN: AP2553.3, R_MOSFET_USB3.2, U2.30
- removed net ZERO_RX: JP2.10, U2.15
- removed net ZERO_TX: JP2.8, U2.16
- new net BTN: R5.2, S1.4, U1.47
- new net N$10: AP1.5, R_MOSFET_USB2.2
- new net N$11: AP2.5, R_MOSFET_USB5.2
- new net N$23: IC3.3, Y2.1
- new net N$24: IC3.2, Y2.3
- new net N$31: IC3.14, REXT.2
- new net N$5: C25.2, U1.43
- new net N$8: C4.2, U1.1, Y1.P$2
- new net UC_DM: IC3.10, U1.33
- new net UC_DP: IC3.11, U1.34
- new net USB0_EN: AP2.3, R_MOSFET_USB6.2, U1.26
- new net USB1_EN: AP2553.3, R_MOSFET_USB3.2, U1.30
- new net USB1_OUT: AP2553.6, C12.2, C2.2, USB_1.VBUS
- new net USB2_EN: AP1.3, R_MOSFET_USB4.2, U1.28
- new net USB2_OUT: AP1.6, C18.2, C20.2, USB_2.VBUS
- new net USB_1_DM: IC3.8, USB_1.D-
- new net USB_1_DP: IC3.9, USB_1.D+
- new net USB_2_DM: IC3.6, USB_2.D-
- new net USB_2_DP: IC3.7, USB_2.D+
- new net USB_3_DM: IC3.4
- new net USB_3_DP: IC3.5
- new net VCC_5V: AP1.1, AP2.1, AP2553.1, C10.1, C11.1, C17.1, C21.1, C22.1, C3.1, C7.1, IC1.2@1, IC3.20
- new net VD_18: C28.1, IC3.12, IC3.28
- new net VD_33: C29.2, IC3.13, IC3.19, IC3.21, IC3.26, R7.2
- new net VD_INT: C6.1, U1.7, VD1.1, VD2.2
- net BATT_VCC: now also J4.PWR, Q3.2, R4.1; no longer C18.1, C5.+, J1.PWR, Q1.2, R9.1
- net CAM_EN: now also R6.1, U1.10; no longer R10.1, U2.47
- net CAM_OUT: now also J3.PWR, Q3.3; no longer J2.PWR, Q1.3
- net CONV_5V: no longer AP2553.1, C17.2, C2.1, C22.1, C7.1, IC2.2@1
- net GND: now also AP1.2, AP2.2, C1.2, C10.2, C11.2, C17.2, C18.1, C2.1, C23.1, C24.1, C25.1, C28.2, C29.1, C3.2, C5.1, IC1.1, IC3.1, J2.3, J2.5, J3.GND, J4.GND, Q4.2, REXT.1, R_MOSFET_USB2.1, R_MOSFET_USB4.1, R_MOSFET_USB5.1, R_MOSFET_USB6.1, S1.2, U1.18, U1.35, U1.42, USB_1.GND, USB_2.GND; no longer C10.1, C11.1, C2.2, C3.1, C5.-, IC1.2, IC1.4, IC2.1, J1.GND, J2.GND, J5.3, J5.5, JP1.1, JP2.6, Q2.2, SW1.P$1, SW2.P$1, U2.18, U2.35, U2.42, U2.5
- net GNDA: now also D1.A; no longer C17.1, C18.2
- net LED: now also U1.27; no longer U2.26
- net MICRO_DM: now also IC3.15; no longer U2.33
- net MICRO_DP: now also IC3.16; no longer U2.34
- net MICRO_VBUS: now also AP2.6, C23.2, C24.2, IC3.18
- net N$15: now also IC3.17, R7.1; no longer IC1.3, R15.2
- net N$2: now also Q4.1, R6.2; no longer C21.1, U2.43
- net N$26: now also D1.C
- net N$3: now also Q3.1, Q4.3, R4.2; no longer C10.2, U2.1, Y2.P$2
- net N$32: now also C5.2, U1.2, Y1.P$1; no longer C11.2, U2.2, Y2.P$1
- net RESET: now also J2.10, U1.40; no longer J5.10, U2.40
- net SCL: now also U1.32; no longer U2.32
- net SDA: now also U1.31; no longer U2.31
- net SWDCLK: now also J2.4, U1.45; no longer J5.4, U2.45
- net SWDIO: now also J2.2, U1.46; no longer J5.2, U2.46
- net VCC: now also C1.1, IC1.3, J2.1, R5.1, U1.17, U1.36, U1.44, U1.6; no longer C12.2, C20.2, IC2.3, J5.1, RBTN.1, RBTN1.1, U2.17, U2.36, U2.44, U2.6
Routing:
- net VD_33: track 0.00 -> 63.0 mm, vias 0 -> 2
- net GND: track 51.0 -> 113.8 mm, vias 10 -> 29
- net VD_18: track 0.00 -> 41.4 mm, vias 0 -> 2
- net VCC_5V: track 0.00 -> 38.9 mm, vias 0 -> 1
- net CONV_5V: track 28.0 -> 0.00 mm, vias 3 -> 0
- net VD_DIRECT: track 27.9 -> 0.00 mm, vias 1 -> 0
- net USB0_EN: track 0.00 -> 22.9 mm, vias 0 -> 1
- net USB2_EN: track 0.00 -> 22.8 mm, vias 0 -> 1
- net ZERO_RX: track 20.2 -> 0.00 mm
- net ZERO_TX: track 19.5 -> 0.00 mm
- net CAM1: track 19.3 -> 0.00 mm, vias 2 -> 0
- net BATT_VCC: track 17.9 -> 36.1 mm, vias 1 -> 0
- net MICRO_VBUS: track 0.00 -> 17.4 mm, vias 0 -> 1
- net CAM2: track 16.9 -> 0.00 mm, vias 2 -> 0
- net CAM_OUT: track 16.1 -> 0.00 mm
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- added copper zone on layer 16, net CAM_OUT
- added copper zone on layer 1, net MICRO_VBUS
- added copper zone on layer 1, net USB1_OUT
- added copper zone on layer 1, net USB2_OUT
- added copper zone on layer 16, net USB2_OUT
- added copper zone on layer 1, net VCC_5V
- removed copper zone on layer 16, net CONV_5V
- removed copper zone on layer 16, net ZERO_5V
Other:
- board text added: "15"
- board text removed: "11"
- board text removed: "5V"
- board text removed: "VD1"
- board text removed: "VD2"

Commit message: batteryholder boards minor changes
Parts:
- C13: device SparkFun-Capacitors:0805 -> SparkFun-Capacitors:1206
- Y2: device SparkFun-FreqCtrl:CRYSTAL-SMD-5X3 -> SparkFun-FreqCtrl:HC49U-V
- moved AP1 2.03 mm to (14.7, 60.7)
- moved C17 1.80 mm to (11.4, 62.7)
- moved Y2 1.48 mm to (14.5, 57.9)
- moved R_MOSFET_USB2 1.44 mm to (14.7, 63.5), turned to 0 degrees
- moved C21 1.02 mm to (10.2, 54.9)
- moved R_MOSFET_USB4 1.02 mm to (15.0, 54.9)
- moved C13 0.72 mm to (16.8, 15.4), flipped to the bottom
- moved C18 0.51 mm to (20.3, 58.9)
- moved C20 0.51 mm to (20.3, 61.5)
- moved C3 0.25 mm to (9.65, 59.9)
Connections:
- net N$24: now also Y2.2; no longer Y2.3
Routing:
- net GND: track 113.8 -> 109.4 mm, vias 29 -> 30
- net VD_18: track 41.4 -> 45.3 mm
- net VD_33: track 63.0 -> 66.3 mm
- net N$23: track 5.44 -> 8.49 mm
- net USB2_EN: track 22.8 -> 24.8 mm
- net VCC_5V: track 38.9 -> 37.7 mm
- net N$26: track 13.3 -> 12.2 mm, vias 2 -> 1
- net N$24: track 7.56 -> 8.58 mm
- net N$11: track 5.21 -> 4.21 mm
- net N$27: track 2.46 -> 1.60 mm, vias 0 -> 1
- net N$10: track 4.71 -> 3.96 mm
Other:
- board text added: "2"

Commit message: cleanup commit (various changes)
Parts:
- added C26: 100uF, SparkFun-Capacitors:1206
- moved C3 1.93 mm to (8.89, 61.7), turned to 90 degrees
- moved R4 1.85 mm to (28.2, 20.6), flipped to the top, turned to 90 degrees
- moved R5 1.02 mm to (26.2, 33.5)
- moved Q4 0.51 mm to (25.4, 20.4)
- moved R6 0.51 mm to (22.4, 20.3)
- moved Y2 0.51 mm to (14.0, 57.9)
- moved C7 0.25 mm to (3.30, 32.0)
- moved C21 0.25 mm to (10.2, 54.6)
Connections:
- net BTN: now also S1.3
- net GND: now also C26.2, R5.1, USB_1.SHLD1, USB_1.SHLD2, USB_2.SHLD1, USB_2.SHLD2; no longer S1.2
- net VCC: now also S1.1, S1.2; no longer R5.1
- net VCC_5V: now also C26.1
Routing:
- net VCC: track 65.7 -> 72.0 mm
- net GND: track 109.4 -> 103.6 mm
- net BTN: track 16.0 -> 21.6 mm
- net CAM_EN: track 18.6 -> 18.0 mm
- net BATT_VCC: track 35.8 -> 35.4 mm, vias 0 -> 1
