File: eagle/controller15_2/controller15_2.sch (EAGLE design)
At the start: 75 parts, among them IC1 MCP170312MB, IC3 FE1.1S, J2 CORTEX_DEBUG_PTH, J3 POWER_JACKPTH_BREAD, J4 POWER_JACKPTH_BREAD, Q3 FDD4141TO252, Q4 200mA/50V, U1 ATSAMD21G-A, U3 MP2307, X2 ZX62D-B-5PA8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

Commit message: batteryholder boards minor changes
Parts:
- C13: device SparkFun-Capacitors:CAP0805 -> SparkFun-Capacitors:CAP1206
- Y2: device SparkFun-FreqCtrl:CRYSTALCRYSTAL-SMD-5X3-12MHZ -> SparkFun-FreqCtrl:CRYSTALHC49UV
Changed lines of the file:
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@@
 <?xml version="1.0" encoding="utf-8"?>
 <!DOCTYPE eagle SYSTEM "eagle.dtd">
-<eagle version="9.5.0">
+<eagle version="9.5.1">
 <drawing>
 <settings>
@@
 <part name="FRAME2" library="frames" deviceset="DINA4_L" device=""/>
 <part name="FRAME3" library="frames" deviceset="A3L-LOC" device=""/>
-<part name="C13" library="SparkFun-Capacitors" deviceset="CAP" device="0805" value="10nF"/>
+<part name="C13" library="SparkFun-Capacitors" deviceset="CAP" device="1206" value="10nF"/>
 <part name="R1" library="SparkFun-Resistors" deviceset="RESISTOR" device="1206" value="6.8k"/>
 <part name="R2" library="SparkFun-Resistors" deviceset="RESISTOR" device="1206" value="10k / 1%"/>
@@
 <part name="USB_2" library="SparkFun-Connectors" library_urn="urn:adsk.eagle:library:513" deviceset="USB_A" device="_SMT_FEMALE" package3d_urn="urn:adsk.eagle:package:38297/1"/>
 <part name="GND23" library="SparkFun-Aesthetics" deviceset="GND" device=""/>
-<part name="Y2" library="SparkFun-FreqCtrl" deviceset="CRYSTAL" device="CRYSTAL-SMD-5X3-12MHZ" value="12MHz"/>
+<part name="Y2" library="SparkFun-FreqCtrl" deviceset="CRYSTAL" device="HC49UV" value="12MHz"/>
 <part name="REXT" library="SparkFun-Passives" deviceset="RESISTOR" device="0805-RES" value="2.7k / 1%"/>
 <part name="GND24" library="SparkFun-Aesthetics" deviceset="GND" device=""/>
@@
 <instance part="Y2" gate="G$1" x="78.74" y="104.14" smashed="yes" rot="R90">
 <attribute name="NAME" x="77.724" y="106.68" size="1.778" layer="95" rot="R90"/>
-<attribute name="VALUE" x="81.28" y="106.68" size="1.778" layer="96" rot="R90"/>
 </instance>
 <instance part="REXT" gate="G$1" x="88.9" y="63.5" smashed="yes" rot="R90">

Commit message: cleanup commit (various changes)
Parts:
- added C26: 100uF, SparkFun-Capacitors:1.0UF-1206-50V-10%
Connections:
- net BTN: now also S1.3
- net GND: now also C26.2, R5.1, USB_1.SHIELD, USB_2.SHIELD; no longer S1.2
- net VCC: now also S1.1, S1.2; no longer R5.1
- net VCC_5V: now also C26.1
Other:
- note added: "(optional)"
