File: eagle/templog3/templog3.brd (EAGLE design)
At the start: 30 x 65 mm, 64 parts, among them IC1 ILD213T, IC2 MCP170312MB, J1 POWER_JACKPTH_BREAD, J2 POWER_JACKPTH_BREAD, J5 CORTEX_DEBUG_PTH, Q2 200mA/50V, SW1 KSS221GLFS, SW2 KSS221GLFS, U2 ATSAMD21G-A, U3 MP2307, X1 1501_04, X2 ZX62D-B-5PA8, Y2 32.768kHz

Commit message: additional eagle boards
Parts:
- removed AP2553: MCP4725, SparkFun-IC-Conversion:SOT23-6
- removed C10, C11: 15pF, SparkFun-Passives:0805
- removed C12, C20, C21, C9: 0.1uF, SparkFun-Capacitors:0805
- removed C13: 10nF, SparkFun-Capacitors:1206
- removed C14: 3.9nF, SparkFun-Capacitors:1206
- removed C15: 0.1uF, SparkFun-Capacitors:1206
- removed C16, C17: 22uF / 6.3V, SparkFun-Capacitors:1210
- removed C18, C19: 10uF / 25V, SparkFun-Capacitors:1210
- removed C22: 120uF, SparkFun-Capacitors:1206
- removed D2: (no value), SparkFun-LED:WS2812B
- removed H1, H2, H3, H4: MOUNT-HOLE2.8, holes:2,8
- removed IC2: MCP170312MB, linear:SOT89
- removed J1: POWER_JACKPTH_BREAD, SparkFun-Connectors:POWER_JACK_PTH_BREAD
- removed J5: CORTEX_DEBUG_PTH, SparkFun-Connectors:2X5-PTH-1.27MM
- removed JP1: (no value), SparkFun-Passives:PAD-JUMPER-2-NO_YES_SILK
- removed JP2: (no value), adafruit:2X20
- removed L2: 10uH / 4A, SparkFun-Passives:SRU1038
- removed Q1: (no value), transistor-fet:TO252
- removed Q2: 200mA/50V, SparkFun-DiscreteSemi:SOT23-3
- removed R1: 6.8k, SparkFun-Resistors:1206
- removed R10: 1k, SparkFun-Resistors:0805
- removed R15, R20: (no value), SparkFun-Passives:0805
- removed R2: 10k / 1%, SparkFun-Resistors:1206
- removed R24: 100K, SparkFun-Resistors:1206
- removed R3: 44k / 1%, SparkFun-Resistors:1206
- removed R9: 10k, SparkFun-Resistors:0805
- removed RBTN, RBTN1, RRST1, R_MOSFET_USB3: 10k, SparkFun-Passives:0805
- removed R_LED: 4.7k, SparkFun-Resistors:0805
- removed R_MOSFET_USB1: ? (1%), SparkFun-Passives:0805
- removed SH2: SHORT-HT5, shorts:SHORT_TOP-50
- removed SW1, SW2: KSS221GLFS, adafruit:BTN_CK_KSS
- removed U2: ATSAMD21G-A, SparkFun-IC-Microcontroller:TQFP-48
- removed U3: MP2307, SparkFun-AnalogIC:SO08
- removed VD1: 10k, SparkFun-Passives:1206
- removed VD2: 6.2k, SparkFun-Passives:1206
- removed X1: 1501_04, con-lumberg:1501_05
- added D1: (no value), SparkFun-LED:LED-1206
- added RRST: 10k, SparkFun-Passives:0805
- added R_I2C_3: 4.7k, SparkFun-Passives:0805
- added R_I2C_4: (no value), SparkFun-Passives:0805
- added TP1, TP2, TP3, TP4, TP5: TPB1,27, testpad:B1,27
- added U$1: MICROSD, adafruit:MICROSD
- added U1: ATSAMD21G-A, SparkFun-IC-Microcontroller:TQFP-48
- C3: value 1.0uF -> 0.1uF
- C4: value 120uF -> 22pF; device SparkFun-Capacitors:1206 -> SparkFun-Passives:0805
- C5: value 100uF -> 22pF; device SparkFun-Capacitors:PANASONIC_D -> SparkFun-Passives:0805
- C6: value 0.1uF -> 1.0uF; device SparkFun-Capacitors:1206 -> SparkFun-Capacitors:0805
- C8: device SparkFun-Capacitors:1206 -> SparkFun-Capacitors:0805
- IC1: value ILD213T -> MCP170312MB; device SparkFun-DiscreteSemi:SO08 -> linear:SOT89
- J2: value POWER_JACKPTH_BREAD -> 3-PIN SMD; device SparkFun-Connectors:POWER_JACK_PTH_BREAD -> SparkFun-Connectors:JST-3-SMD
- moved C5 34.8 mm to (18.8, 9.27)
- moved X2 30.0 mm to (0.00, 13.2), turned to 0 degrees
- moved J2 29.3 mm to (25.4, 5.84), turned to 180 degrees
- moved C8 27.7 mm to (6.35, 6.10), flipped to the bottom
- moved C7 24.7 mm to (2.29, 5.84), flipped to the bottom, turned to 180 degrees
- moved C6 23.4 mm to (11.2, 6.60), flipped to the top
- moved IC1 21.9 mm to (3.81, 5.84), turned to 90 degrees
- moved Y2 13.5 mm to (18.5, 6.60), turned to 270 degrees
- moved R_I2C_1 12.6 mm to (20.8, 13.2), flipped to the top, turned to 90 degrees
- moved C3 12.6 mm to (19.1, 12.2), flipped to the top, turned to 90 degrees
- moved MCP9808 12.2 mm to (21.1, 16.8), flipped to the top, turned to 270 degrees
- moved R_I2C_2 11.1 mm to (23.4, 14.2), flipped to the top, turned to 0 degrees
- moved C4 8.08 mm to (16.6, 6.60), flipped to the top, turned to 90 degrees
- moved C2 7.06 mm to (14.2, 6.60), flipped to the top
Connections:
- removed net BATT_VCC: C18.1, C19.2, C5.+, J1.PWR, Q1.2, R24.1, R9.1, U3.2, VD1.2
- removed net BTN1: RBTN.2, SW1.P$2, U2.24
- removed net BTN2: RBTN1.2, SW2.P$2, U2.25
- removed net CAM1: R20.1, U2.10
- removed net CAM2: R15.1, U2.11
- removed net CAM_EN: R10.1, U2.47
- removed net CAM_OUT: J2.PWR, Q1.3
- removed net CONV_5V: AP2553.1, C16.2, C17.2, C2.1, C22.1, C7.1, IC2.2@1, L2.1, R3.2
- removed net GNDA: C15.1, C16.1, C17.1, C18.2, C19.1, R1.2, R2.2, SH2.1, U3.4, U3.BTM, U3.P$1
- removed net N$12: IC1.6, X1.2
- removed net N$13: IC1.8, X1.3
- removed net N$15: IC1.3, R15.2
- removed net N$19: IC1.1, R20.2
- removed net N$2: C21.1, U2.43
- removed net N$25: C15.2, U3.8
- removed net N$26: C13.2, L2.2, U3.3
- removed net N$27: C13.1, U3.1
- removed net N$28: C14.1, R1.1
- removed net N$29: C14.2, U3.6
- removed net N$3: C10.2, U2.1, Y2.P$2
- removed net N$30: R2.1, R3.1, U3.5
- removed net N$34: IC1.5, IC1.7, JP1.2, X1.1
- removed net N$4 (its old number): AP2553.5, R_MOSFET_USB1.2
- removed net N$6: Q2.1, R10.2
- removed net N$7: D2.4, R_LED.2
- removed net PB_BUCK_EN: R24.2, U3.7
- removed net USB_FAULT: U2.38
- removed net VD_DIRECT: C6.1, U2.12, VD1.1, VD2.2
- removed net ZERO_5V: AP2553.6, C3.2, C4.2, JP2.2
- removed net ZERO_EN: AP2553.3, R_MOSFET_USB3.2, U2.30
- removed net ZERO_RX: JP2.10, U2.15
- removed net ZERO_TX: JP2.8, U2.16
- new net CD: U$1.CD1, U1.24
- new net CS: U$1.2, U1.27
- new net EXT_SENSOR: J2.2, R_I2C_3.1, U1.14
- new net MISO: U$1.7, U1.28
- new net MOSI: U$1.3, U1.25
- new net N$5: D1.C, R_I2C_4.1
- new net N$8: C4.2, U1.1, Y2.P$2
- new net SCK: U$1.5, U1.26
- net GND: now also C2.1, C5.1, IC1.1, J2.3, TP5.TP, U$1.6, U$1.MT1, U$1.MT2, U1.18, U1.35, U1.42, U1.5; no longer AP2553.2, C10.1, C11.1, C12.1, C2.2, C20.1, C21.2, C22.2, C5.-, C9.2, D2.3, IC1.2, IC1.4, IC2.1, J1.GND, J2.GND, J5.3, J5.5, JP1.1, JP2.6, Q2.2, R_MOSFET_USB1.1, R_MOSFET_USB3.1, SH2.2, SW1.P$1, SW2.P$1, U2.18, U2.35, U2.42, U2.5, VD2.1
- net LED: now also R_I2C_4.2, U1.48; no longer R_LED.1, U2.26
- net MICRO_DM: now also U1.33; no longer U2.33
- net MICRO_DP: now also U1.34; no longer U2.34
- net MICRO_VBUS: now also C7.1, IC1.2@1
- net N$1: now also C6.1, U1.43; no longer Q1.1, Q2.3, R9.2
- net N$32: now also C5.2, U1.2; no longer C11.2, U2.2
- net RESET: now also RRST.1, TP3.TP, U1.40; no longer J5.10, RRST1.1, U2.40
- net SCL: now also U1.32; no longer U2.32
- net SDA: now also U1.31; no longer U2.31
- net SWDCLK: now also TP2.TP, U1.45; no longer J5.4, U2.45
- net SWDIO: now also TP1.TP, U1.46; no longer J5.2, U2.46
- net VCC: now also C2.2, C3.2, D1.A, IC1.3, J2.1, RRST.2, R_I2C_3.2, TP4.TP, U$1.4, U1.17, U1.36, U1.44, U1.6; no longer C12.2, C20.2, C9.1, D2.1, IC2.3, J5.1, RBTN.1, RBTN1.1, RRST1.2, U2.17, U2.36, U2.44, U2.6
Routing:
- net CONV_5V: track 28.0 -> 0.00 mm, vias 3 -> 0
- net VD_DIRECT: track 27.9 -> 0.00 mm, vias 1 -> 0
- net CS: track 0.00 -> 22.9 mm, vias 0 -> 1
- net EXT_SENSOR: track 0.00 -> 22.5 mm, vias 0 -> 2
- net MOSI: track 0.00 -> 21.1 mm, vias 0 -> 1
- net CAM_EN: track 20.6 -> 0.00 mm, vias 1 -> 0
- net ZERO_RX: track 20.2 -> 0.00 mm
- net LED: track 5.12 -> 24.9 mm, vias 1 -> 2
- net ZERO_TX: track 19.5 -> 0.00 mm
- net CAM1: track 19.3 -> 0.00 mm, vias 2 -> 0
- net SWDIO: track 24.3 -> 5.28 mm, vias 1 -> 0
- net SCK: track 0.00 -> 18.4 mm, vias 0 -> 1
- net BATT_VCC: track 17.9 -> 0.00 mm, vias 1 -> 0
- net VCC: track 77.2 -> 59.8 mm, vias 8 -> 2
- net N$30: track 17.4 -> 0.00 mm, vias 2 -> 0
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- added copper zone on layer 1, net MICRO_VBUS
- added copper zone on layer 16, net MICRO_VBUS
- removed copper zone on layer 1, net BATT_VCC
- removed copper zone on layer 16, net BATT_VCC
- removed copper zone on layer 1, net CONV_5V
- removed copper zone on layer 16, net CONV_5V
- removed copper zone on layer 1, net GNDA
- removed copper zone on layer 16, net GNDA
- removed copper zone on layer 1, net N$26
- removed copper zone on layer 16, net ZERO_5V
Other:
- board size 30 x 65 mm -> 31.2 x 16 mm
- board text added: "TEMPlog3"
- board text removed: "11"
- board text removed: "5V"
- board text removed: "BOX"
- board text removed: "IN"
- board text removed: "OUT"
- board text removed: "TIME"
- board text removed: "VD1"
- board text removed: "VD2"

Commit message: batteryholder boards minor changes
Parts:
- moved J2 4.43 mm to (28.3, 9.20), turned to 270 degrees
- moved R_I2C_3 1.08 mm to (25.9, 15.7), turned to 180 degrees
- moved R_I2C_4 0.80 mm to (29.2, 15.7), turned to 180 degrees
- moved C6 0.25 mm to (10.9, 6.60)
- moved R_I2C_1 0.25 mm to (20.8, 13.5)
- moved C5 0.14 mm to (18.7, 9.37)
Routing:
- net VCC: track 59.8 -> 45.6 mm
- net EXT_SENSOR: track 22.5 -> 28.1 mm
- net GND: track 34.0 -> 38.0 mm, vias 9 -> 11
- net LED: track 24.9 -> 22.6 mm
Other:
- board size 31.2 x 16 mm -> 31 x 16 mm
- board text added: "DAT"
- board text added: "DS18S20"
- board text added: "EXT."
- board text added: "GND"
- board text added: "SENSOR"
- board text added: "VCC"
