File: eagle/BMS_breakout_2/BMS_breakout_2.brd (EAGLE design)
At the start: 71 x 24 mm, 14 parts, among them J4 5.5x2.1mm Barrel

Commit message: eagle: BMS breakout 2
Parts:
- removed J8: (no value), SparkFun-Connectors:2X3-SHROUDED
- removed X1: (no value), con-molex-micro-fit-3_0:43650-0309
- removed X2: (no value), con-molex-micro-fit-3_0:43045-0600
- moved J3 12.0 mm to (67.8, 7.02)
Connections:
- net B+: no longer J8.1, J8.2
- net B-: no longer J8.5, J8.6
- net BM: no longer J8.3, J8.4
Routing:
- net BM: track 9.97 -> 11.0 mm
Changed lines of the file:
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@@
 </autorouter>
 <elements>
-<element name="J3" library="SparkFun-Connectors" library_urn="urn:adsk.eagle:library:513" package="SCREWTERMINAL-5MM-3" package3d_urn="urn:adsk.eagle:package:38070/1" value="" x="79.77" y="6.62" smashed="yes" rot="R90">
-<attribute name="PROD_ID" value="CONN-10134" x="79.77" y="6.62" size="1.778" layer="27" rot="R90" display="off"/>
-<attribute name="SF_SKU" value="PRT-08433" x="79.77" y="6.62" size="1.778" layer="27" rot="R90" display="off"/>
-<attribute name="VALUE" x="77.865" y="10.049" size="0.6096" layer="27" font="vector" ratio="20" rot="R90"/>
+<element name="J3" library="SparkFun-Connectors" library_urn="urn:adsk.eagle:library:513" package="SCREWTERMINAL-5MM-3" package3d_urn="urn:adsk.eagle:package:38070/1" value="" x="67.77" y="7.02" smashed="yes" rot="R90">
+<attribute name="PROD_ID" value="CONN-10134" x="67.77" y="7.02" size="1.778" layer="27" rot="R90" display="off"/>
+<attribute name="SF_SKU" value="PRT-08433" x="67.77" y="7.02" size="1.778" layer="27" rot="R90" display="off"/>
+<attribute name="VALUE" x="65.865" y="10.449" size="0.6096" layer="27" font="vector" ratio="20" rot="R90"/>
 </element>
 <element name="J4" library="SparkFun-Connectors" library_urn="urn:adsk.eagle:library:513" package="POWER_JACK_SMD" package3d_urn="urn:adsk.eagle:package:38221/1" value="5.5x2.1mm Barrel" x="2.5" y="12" smashed="yes">
@@
 <attribute name="POPULARITY" value="7" x="65" y="0" size="1.778" layer="27" display="off"/>
 </element>
-<element name="X1" library="con-molex-micro-fit-3_0" package="43650-0309" value="" x="89" y="42" smashed="yes" rot="R90"/>
 <element name="H1" library="holes" library_urn="urn:adsk.eagle:library:237" package="3,2" package3d_urn="urn:adsk.eagle:package:14275/1" value="MOUNT-HOLE3.2" x="65" y="24" smashed="yes">
 <attribute name="POPULARITY" value="7" x="65" y="24" size="1.778" layer="27" display="off"/>
 </element>
-<element name="J8" library="SparkFun-Connectors" library_urn="urn:adsk.eagle:library:513" package="2X3-SHROUDED" package3d_urn="urn:adsk.eagle:package:38264/1" value="" x="65.5" y="12" smashed="yes">
-<attribute name="PROD_ID" value="CONN-10681" x="65.5" y="12" size="1.778" layer="27" display="off"/>
-<attribute name="SF_ID" value="PRT_10877" x="65.5" y="12" size="1.778" layer="27" display="off"/>
-<attribute name="VALUE" x="61.69" y="3.618" size="0.6096" layer="27" font="vector" ratio="20"/>
-</element>
-<element name="X2" library="con-molex-micro-fit-3_0" package="43045-0600" value="" x="94" y="12" smashed="yes" rot="R90"/>
 </elements>
 <signals>
@@
 <contactref element="J3" pad="3"/>
 <contactref element="J1" pad="1"/>
-<contactref element="J8" pad="1"/>
-<contactref element="J8" pad="2"/>
-<wire x1="66.77" y1="14.54" x2="64.23" y2="14.54" width="2" layer="16"/>
-<wire x1="64.23" y1="14.54" x2="62.46" y2="14.54" width="2" layer="16"/>
-<wire x1="62.46" y1="14.54" x2="56.8" y2="20.2" width="2" layer="16"/>
-<wire x1="66.77" y1="14.54" x2="79.77" y2="16.62" width="0" layer="19" extent="1-1"/>
+<wire x1="67.77" y1="17.02" x2="59.98" y2="17.02" width="3" layer="16"/>
+<wire x1="59.98" y1="17.02" x2="56.8" y2="20.2" width="3" layer="16"/>
 </signal>
 <signal name="BM">
@@
 <contactref element="J3" pad="2"/>
 <contactref element="J2" pad="1"/>
-<contactref element="J8" pad="4"/>
-<contactref element="J8" pad="3"/>
-<wire x1="56.8" y1="12" x2="64.23" y2="12" width="2" layer="16"/>
-<wire x1="64.23" y1="12" x2="66.77" y2="12" width="2" layer="16"/>
-<wire x1="66.77" y1="12" x2="79.77" y2="11.62" width="0" layer="19" extent="1-1"/>
+<wire x1="67.77" y1="12.02" x2="56.82" y2="12.02" width="3" layer="16"/>
+<wire x1="56.82" y1="12.02" x2="56.8" y2="12" width="3" layer="16"/>
 </signal>
 <signal name="B-">
@@
 <contactref element="J3" pad="1"/>
 <contactref element="J5" pad="1"/>
-<contactref element="J8" pad="6"/>
-<contactref element="J8" pad="5"/>
-<wire x1="66.77" y1="9.46" x2="64.23" y2="9.46" width="2" layer="16"/>
-<wire x1="64.23" y1="9.46" x2="62.46" y2="9.46" width="2" layer="16"/>
-<wire x1="62.46" y1="9.46" x2="56.8" y2="3.8" width="2" layer="16"/>
-<wire x1="66.77" y1="9.46" x2="79.77" y2="6.62" width="0" layer="19" extent="1-1"/>
+<wire x1="67.77" y1="7.02" x2="60.02" y2="7.02" width="3" layer="16"/>
+<wire x1="60.02" y1="7.02" x2="56.8" y2="3.8" width="3" layer="16"/>
 </signal>
 </signals>
