File: eagle/BMS_breakout_2/BMS_breakout_2.sch (EAGLE design)
At the start: 13 parts, among them J4 5.5x2.1mm Barrel

Commit message: eagle: BMS breakout 2
Parts:
- removed J8: (no value), SparkFun-Connectors:CONN_03X2SHROUD
- removed X1: (no value), con-molex-micro-fit-3_0:HEADER_POS3_43650-0309
- removed X2: (no value), con-molex-micro-fit-3_0:HEADER_POS6_43045-0600
Connections:
- net B+: no longer J8.1, J8.2
- net B-: no longer J8.5, J8.6
- net BM: no longer J8.3, J8.4
Changed lines of the file:
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@@
 <part name="H3" library="holes" library_urn="urn:adsk.eagle:library:237" deviceset="MOUNT-HOLE" device="3.2" package3d_urn="urn:adsk.eagle:package:14275/1"/>
 <part name="H4" library="holes" library_urn="urn:adsk.eagle:library:237" deviceset="MOUNT-HOLE" device="3.2" package3d_urn="urn:adsk.eagle:package:14275/1"/>
-<part name="X1" library="con-molex-micro-fit-3_0" deviceset="HEADER_POS3_?" device="43650-0309"/>
-<part name="J8" library="SparkFun-Connectors" library_urn="urn:adsk.eagle:library:513" deviceset="CONN_03X2" device="SHROUD" package3d_urn="urn:adsk.eagle:package:38264/1"/>
-<part name="X2" library="con-molex-micro-fit-3_0" deviceset="HEADER_POS6_?" device="43045-0600"/>
 </parts>
 <sheets>
@@
 <attribute name="VALUE" x="118.872" y="71.1962" size="1.778" layer="96"/>
 </instance>
-<instance part="X1" gate="G$1" x="22.86" y="91.44" smashed="yes" rot="R180">
-<attribute name="VALUE" x="24.13" y="99.06" size="1.778" layer="96" rot="R180"/>
-<attribute name="NAME" x="24.13" y="85.598" size="1.778" layer="95" rot="R180"/>
-</instance>
-<instance part="J8" gate="G$1" x="22.86" y="63.5" smashed="yes">
-<attribute name="NAME" x="19.304" y="69.088" size="1.778" layer="95" font="vector"/>
-<attribute name="VALUE" x="19.558" y="57.658" size="1.778" layer="96" font="vector" align="top-left"/>
-</instance>
-<instance part="X2" gate="G$1" x="50.8" y="104.14" smashed="yes">
-<attribute name="VALUE" x="49.53" y="93.98" size="1.778" layer="96"/>
-<attribute name="NAME" x="49.53" y="115.062" size="1.778" layer="95"/>
-</instance>
 </instances>
 <busses>
@@
 <wire x1="53.34" y1="78.74" x2="73.66" y2="78.74" width="0.1524" layer="91"/>
 <label x="66.04" y="81.28" size="1.778" layer="95"/>
-<pinref part="J8" gate="G$1" pin="1"/>
-<pinref part="J8" gate="G$1" pin="2"/>
-<wire x1="15.24" y1="66.04" x2="30.48" y2="66.04" width="0.1524" layer="91"/>
-<wire x1="30.48" y1="66.04" x2="43.18" y2="66.04" width="0.1524" layer="91"/>
-<junction x="30.48" y="66.04"/>
-<junction x="43.18" y="66.04"/>
 </segment>
 </net>
@@
 <pinref part="J2" gate="G$1" pin="1"/>
 <label x="66.04" y="66.04" size="1.778" layer="95"/>
-<pinref part="J8" gate="G$1" pin="4"/>
-<wire x1="43.18" y1="63.5" x2="30.48" y2="63.5" width="0.1524" layer="91"/>
-<junction x="43.18" y="63.5"/>
-<pinref part="J8" gate="G$1" pin="3"/>
-<wire x1="30.48" y1="63.5" x2="15.24" y2="63.5" width="0.1524" layer="91"/>
-<junction x="30.48" y="63.5"/>
 </segment>
 </net>
@@
 <pinref part="J5" gate="G$1" pin="1"/>
 <label x="66.04" y="53.34" size="1.778" layer="95"/>
-<pinref part="J8" gate="G$1" pin="6"/>
-<wire x1="30.48" y1="60.96" x2="43.18" y2="60.96" width="0.1524" layer="91"/>
-<junction x="43.18" y="60.96"/>
-<pinref part="J8" gate="G$1" pin="5"/>
-<wire x1="30.48" y1="60.96" x2="15.24" y2="60.96" width="0.1524" layer="91"/>
-<junction x="30.48" y="60.96"/>
 </segment>
 </net>
