File: eagle/controller15_3/controller15_3.brd (EAGLE design)
At the start: 30 x 65 mm, 81 parts, among them IC1 MCP1703AT, IC2 ILD213T, IC3 FE1.1S, J2 CORTEX_DEBUG_PTH, J3 POWER_JACKPTH_BREAD, J4 POWER_JACKPTH_BREAD, Q4 200mA/50V, U1 ATSAMD21G-A, U3 MP2307, X1 1501_04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

Commit message: various uncommitted files
Parts:
- VD1: value 10k -> 100k
- VD2: value 6.2k -> 62k
Changed lines of the file:
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@@
 </autorouter>
 <elements>
-<element name="VD1" library="SparkFun-Passives" package="1206" value="10k" x="17.018" y="21.209" smashed="yes" rot="R270"/>
-<element name="VD2" library="SparkFun-Passives" package="1206" value="6.2k" x="14.732" y="21.209" smashed="yes" rot="R90"/>
+<element name="VD1" library="SparkFun-Passives" package="1206" value="100k" x="17.018" y="21.209" smashed="yes" rot="R270"/>
+<element name="VD2" library="SparkFun-Passives" package="1206" value="62k" x="14.732" y="21.209" smashed="yes" rot="R90"/>
 <element name="C4" library="SparkFun-Passives" package="0805" value="22pF" x="15.621" y="22.606" smashed="yes" rot="MR90"/>
 <element name="C5" library="SparkFun-Passives" package="0805" value="22pF" x="12.827" y="22.606" smashed="yes" rot="MR90"/>
