File: eagle/zerocam2S_revD/zerocam2S_revD.brd (EAGLE design)
At the start: 30 x 65 mm, 60 parts, among them IC1 MCP170312MB, J5 CORTEX_DEBUG_PTH, SW1 KSS221GLFS, U1 ATSAMD21G-A, U3 MP2307, X2 ZX62D-B-5PA8, Y2 32.768kHz

Commit message: various uncommitted files
Parts:
- added X1: 2060-1402/998-404, con-wago_2060:P-2060-1402/998-404
- moved C8 4.22 mm to (9.50, 12.8), flipped to the bottom, turned to 90 degrees
- moved R24 4.04 mm to (9.50, 7.38), flipped to the bottom, turned to 270 degrees
- moved JP1 3.10 mm to (21.2, 4.40), turned to 180 degrees
- moved J1 1.72 mm to (13.2, 4.88)
- moved D2 1.40 mm to (26.4, 35.6)
- moved C7 1.33 mm to (20.3, 11.9), turned to 270 degrees
Connections:
- net BATT_VCC: now also X1.L2.1, X1.L2.2
- net GNDA: now also X1.L1.1, X1.L1.2
Routing:
- net BATT_VCC: track 49.2 -> 56.1 mm
- net PB_BUCK_EN: track 39.1 -> 44.1 mm
- net GNDA: track 19.0 -> 14.1 mm
- net VCC: track 92.7 -> 96.2 mm
- net N$27: track 4.78 -> 2.06 mm
- net LED: track 21.4 -> 20.0 mm
- net GND: track 69.2 -> 67.9 mm
- net USB_FAULT: track 9.70 -> 10.9 mm
- net N$25: track 4.14 -> 4.90 mm, vias 0 -> 1
Other:
- outline, holes or cut-outs redrawn
- board text added: "ON"
- board text added: "rev. D"
- board text removed: "OFF"
- board text removed: "rev. E"
